File: schematics/KPNN2024/Board/RADIO.sch (EAGLE design)
At the start: 1 part

Commit message: Даня верни клей
Parts:
- added J1, J2: U.FL-R-SMT-1_10_, UNKNOWN-2024:U.FL-R-SMT-1_10_
- added U$2: NRF24L01_ML01SP4, UNKNOWN-2024:NRF24L01_ML01SP4
- added U$3: XQ-02A, UNKNOWN-2024:XQ-02A
Connections:
- new net 3V3: U$1.UCC, U$2.VCC, U$3.3.3V
- new net 5V: U$3.5V
- new net ATN_RADIO: J2.3, U$3.ANT
- new net CE: U$2.CE
- new net CSN: U$2.CSN
- new net GND: J1.1, J1.2, J2.1, J2.2, U$1.GND, U$2.GND, U$3.GND
- new net IRQ: U$2.IRQ
- new net MISO: U$2.MISO
- new net MOSI: U$2.MOSI
- new net N$2: U$3.LED2
- new net N$3: U$3.LED1
- new net RF-IN: J1.3, U$3.RF-IN
- new net RX: U$1.RX
- new net SCK: U$2.SCK
- new net SW: U$3.SW
- new net TX: U$1.TX
Changed lines of the file:
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@@
 <parts>
 <part name="U$1" library="UNKNOWN-2024" deviceset="GPS-NEO7M" device=""/>
+<part name="U$2" library="UNKNOWN-2024" deviceset="NRF24L01_ML01SP4" device=""/>
+<part name="U$3" library="UNKNOWN-2024" deviceset="XQ-02A" device=""/>
+<part name="J1" library="UNKNOWN-2024" deviceset="U.FL-R-SMT-1_10_" device=""/>
+<part name="J2" library="UNKNOWN-2024" deviceset="U.FL-R-SMT-1_10_" device=""/>
 </parts>
 <sheets>
@@
 <attribute name="NAME" x="0" y="89.662" size="1.778" layer="95"/>
 </instance>
+<instance part="U$2" gate="G$1" x="7.62" y="53.34" smashed="yes" rot="R180">
+<attribute name="NAME" x="17.78" y="40.64" size="2.032" layer="95" rot="R180"/>
+</instance>
+<instance part="U$3" gate="G$1" x="86.36" y="78.74" smashed="yes">
+<attribute name="NAME" x="73.66" y="93.98" size="2.54" layer="94"/>
+</instance>
+<instance part="J1" gate="G$1" x="71.12" y="33.02" smashed="yes">
+<attribute name="NAME" x="87.63" y="43.18" size="1.778" layer="95" align="center-left"/>
+<attribute name="VALUE" x="87.63" y="40.64" size="1.778" layer="96" align="center-left"/>
+</instance>
+<instance part="J2" gate="G$1" x="119.38" y="43.18" smashed="yes">
+<attribute name="NAME" x="135.89" y="53.34" size="1.778" layer="95" align="center-left"/>
+<attribute name="VALUE" x="135.89" y="50.8" size="1.778" layer="96" align="center-left"/>
+</instance>
 </instances>
 <busses>
 </busses>
 <nets>
+<net name="GND" class="0">
+<segment>
+<pinref part="U$2" gate="G$1" pin="GND"/>
+<wire x1="20.32" y1="60.96" x2="38.1" y2="60.96" width="0.1524" layer="91"/>
+<label x="33.02" y="60.96" size="1.778" layer="95"/>
+</segment>
+<segment>
+<pinref part="U$1" gate="G$1" pin="GND"/>
+<wire x1="20.32" y1="81.28" x2="27.94" y2="81.28" width="0.1524" layer="91"/>
+<label x="25.4" y="81.28" size="1.778" layer="95"/>
+</segment>
+<segment>
+<pinref part="U$3" gate="G$1" pin="GND"/>
+<wire x1="68.58" y1="83.82" x2="50.8" y2="83.82" width="0.1524" layer="91"/>
+<label x="50.8" y="83.82" size="1.778" layer="95"/>
+</segment>
+<segment>
+<pinref part="J1" gate="G$1" pin="1"/>
+<wire x1="71.12" y1="33.02" x2="55.88" y2="33.02" width="0.1524" layer="91"/>
+<pinref part="J1" gate="G$1" pin="2"/>
+<wire x1="91.44" y1="33.02" x2="91.44" y2="27.94" width="0.1524" layer="91"/>
+<wire x1="91.44" y1="27.94" x2="71.12" y2="27.94" width="0.1524" layer="91"/>
+<wire x1="71.12" y1="27.94" x2="71.12" y2="33.02" width="0.1524" layer="91"/>
+<junction x="71.12" y="33.02"/>
+<label x="55.88" y="33.02" size="1.778" layer="95"/>
+</segment>
+<segment>
+<pinref part="J2" gate="G$1" pin="2"/>
+<wire x1="139.7" y1="43.18" x2="139.7" y2="38.1" width="0.1524" layer="91"/>
+<wire x1="139.7" y1="38.1" x2="119.38" y2="38.1" width="0.1524" layer="91"/>
+<pinref part="J2" gate="G$1" pin="1"/>
+<wire x1="119.38" y1="38.1" x2="119.38" y2="43.18" width="0.1524" layer="91"/>
+<wire x1="119.38" y1="43.18" x2="106.68" y2="43.18" width="0.1524" layer="91"/>
+<junction x="119.38" y="43.18"/>
+<label x="106.68" y="43.18" size="1.778" layer="95"/>
+</segment>
+</net>
+<net name="3V3" class="0">
+<segment>
+<pinref part="U$2" gate="G$1" pin="VCC"/>
+<wire x1="20.32" y1="43.18" x2="38.1" y2="43.18" width="0.1524" layer="91"/>
+<label x="33.02" y="43.18" size="1.778" layer="95"/>
+</segment>
+<segment>
+<pinref part="U$1" gate="G$1" pin="UCC"/>
+<wire x1="20.32" y1="83.82" x2="27.94" y2="83.82" width="0.1524" layer="91"/>
+<label x="25.4" y="83.82" size="1.778" layer="95"/>
+</segment>
+<segment>
+<pinref part="U$3" gate="G$1" pin="3.3V"/>
+<wire x1="68.58" y1="73.66" x2="50.8" y2="73.66" width="0.1524" layer="91"/>
+<label x="50.8" y="73.66" size="1.778" layer="95"/>
+</segment>
+</net>
+<net name="IRQ" class="0">
+<segment>
+<pinref part="U$2" gate="G$1" pin="IRQ"/>
+<wire x1="20.32" y1="58.42" x2="38.1" y2="58.42" width="0.1524" layer="91"/>
+<label x="33.02" y="58.42" size="1.778" layer="95"/>
+</segment>
+</net>
+<net name="MISO" class="0">
+<segment>
+<pinref part="U$2" gate="G$1" pin="MISO"/>
+<wire x1="20.32" y1="55.88" x2="38.1" y2="55.88" width="0.1524" layer="91"/>
+<label x="33.02" y="55.88" size="1.778" layer="95"/>
+</segment>
+</net>
+<net name="MOSI" class="0">
+<segment>
+<pinref part="U$2" gate="G$1" pin="MOSI"/>
+<wire x1="20.32" y1="53.34" x2="38.1" y2="53.34" width="0.1524" layer="91"/>
+<label x="33.02" y="53.34" size="1.778" layer="95"/>
+</segment>
+</net>
+<net name="SCK" class="0">
+<segment>
+<pinref part="U$2" gate="G$1" pin="SCK"/>
+<wire x1="20.32" y1="50.8" x2="38.1" y2="50.8" width="0.1524" layer="91"/>
+<label x="33.02" y="50.8" size="1.778" layer="95"/>
+</segment>
+</net>
+<net name="CSN" class="0">
+<segment>
+<pinref part="U$2" gate="G$1" pin="CSN"/>
+<wire x1="20.32" y1="48.26" x2="38.1" y2="48.26" width="0.1524" layer="91"/>
+<label x="33.02" y="48.26" size="1.778" layer="95"/>
+</segment>
+</net>
+<net name="CE" class="0">
+<segment>
+<pinref part="U$2" gate="G$1" pin="CE"/>
+<wire x1="20.32" y1="45.72" x2="38.1" y2="45.72" width="0.1524" layer="91"/>
+<label x="33.02" y="45.72" size="1.778" layer="95"/>
+</segment>
+</net>
+<net name="TX" class="0">
+<segment>
+<pinref part="U$1" gate="G$1" pin="TX"/>
+<wire x1="20.32" y1="78.74" x2="27.94" y2="78.74" width="0.1524" layer="91"/>
+<label x="25.4" y="78.74" size="1.778" layer="95"/>
+</segment>
+</net>
+<net name="RX" class="0">
+<segment>
+<pinref part="U$1" gate="G$1" pin="RX"/>
+<wire x1="20.32" y1="76.2" x2="27.94" y2="76.2" width="0.1524" layer="91"/>
+<label x="25.4" y="76.2" size="1.778" layer="95"/>
+</segment>
+</net>
+<net name="5V" class="0">
+<segment>
+<pinref part="U$3" gate="G$1" pin="5V"/>
+<wire x1="68.58" y1="78.74" x2="50.8" y2="78.74" width="0.1524" layer="91"/>
+<label x="50.8" y="78.74" size="1.778" layer="95"/>
+</segment>
+</net>
+<net name="N$2" class="0">
+<segment>
+<pinref part="U$3" gate="G$1" pin="LED2"/>
+<wire x1="104.14" y1="83.82" x2="129.54" y2="83.82" width="0.1524" layer="91"/>
+</segment>
+</net>
+<net name="N$3" class="0">
+<segment>
+<pinref part="U$3" gate="G$1" pin="LED1"/>
+<wire x1="104.14" y1="78.74" x2="129.54" y2="78.74" width="0.1524" layer="91"/>
+</segment>
+</net>
+<net name="SW" class="0">
+<segment>
+<pinref part="U$3" gate="G$1" pin="SW"/>
+<wire x1="104.14" y1="73.66" x2="129.54" y2="73.66" width="0.1524" layer="91"/>
+<label x="127" y="73.66" size="1.778" layer="95"/>
+</segment>
+</net>
+<net name="RF-IN" class="0">
+<segment>
+<pinref part="J1" gate="G$1" pin="3"/>
+<wire x1="81.28" y1="43.18" x2="68.58" y2="43.18" width="0.1524" layer="91"/>
+<label x="68.58" y="43.18" size="1.778" layer="95"/>
+</segment>
+<segment>
+<pinref part="U$3" gate="G$1" pin="RF-IN"/>
+<wire x1="104.14" y1="68.58" x2="129.54" y2="68.58" width="0.1524" layer="91"/>
+<label x="124.46" y="68.58" size="1.778" layer="95"/>
+</segment>
+</net>
+<net name="ATN_RADIO" class="0">
+<segment>
+<pinref part="J2" gate="G$1" pin="3"/>
+<wire x1="129.54" y1="53.34" x2="111.76" y2="53.34" width="0.1524" layer="91"/>
+<label x="111.76" y="53.34" size="1.778" layer="95"/>
+</segment>
+<segment>
+<pinref part="U$3" gate="G$1" pin="ANT"/>
+<wire x1="104.14" y1="88.9" x2="129.54" y2="88.9" width="0.1524" layer="91"/>
+<label x="116.84" y="88.9" size="1.778" layer="95"/>
+</segment>
+</net>
 </nets>
 </sheet>

Commit message: Вабба Лабба Даб Даб
Parts:
- added U$4, U$5: CONNECT_3, UNKNOWN-2024:CONNECT_3
Connections:
- removed net N$2: U$3.LED2
- removed net N$3: U$3.LED1
- new net LED1: U$3.LED1, U$4.PIN
- new net LED2: U$3.LED2, U$5.PIN
- net 3V3: now also U$4.P$1, U$5.P$1
- net GND: now also U$4.P$3, U$5.P$3
Changed lines of the file:
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@@
 <part name="J1" library="UNKNOWN-2024" deviceset="U.FL-R-SMT-1_10_" device=""/>
 <part name="J2" library="UNKNOWN-2024" deviceset="U.FL-R-SMT-1_10_" device=""/>
+<part name="U$4" library="UNKNOWN-2024" deviceset="CONNECT_3" device=""/>
+<part name="U$5" library="UNKNOWN-2024" deviceset="CONNECT_3" device=""/>
 </parts>
 <sheets>
@@
 <attribute name="VALUE" x="135.89" y="50.8" size="1.778" layer="96" align="center-left"/>
 </instance>
+<instance part="U$4" gate="G$1" x="187.96" y="71.12" smashed="yes">
+<attribute name="NAME" x="187.96" y="78.74" size="1.778" layer="94"/>
+</instance>
+<instance part="U$5" gate="G$1" x="187.96" y="86.36" smashed="yes">
+<attribute name="NAME" x="187.96" y="93.98" size="1.778" layer="94"/>
+</instance>
 </instances>
 <busses>
@@
 <label x="106.68" y="43.18" size="1.778" layer="95"/>
 </segment>
+<segment>
+<pinref part="U$5" gate="G$1" pin="P$3"/>
+<wire x1="182.88" y1="88.9" x2="170.18" y2="88.9" width="0.1524" layer="91"/>
+<label x="170.18" y="88.9" size="1.778" layer="95"/>
+</segment>
+<segment>
+<pinref part="U$4" gate="G$1" pin="P$3"/>
+<wire x1="182.88" y1="73.66" x2="170.18" y2="73.66" width="0.1524" layer="91"/>
+<label x="170.18" y="73.66" size="1.778" layer="95"/>
+</segment>
 </net>
 <net name="3V3" class="0">
@@
 <label x="50.8" y="73.66" size="1.778" layer="95"/>
 </segment>
+<segment>
+<pinref part="U$5" gate="G$1" pin="P$1"/>
+<wire x1="182.88" y1="83.82" x2="170.18" y2="83.82" width="0.1524" layer="91"/>
+<label x="170.18" y="83.82" size="1.778" layer="95"/>
+</segment>
+<segment>
+<pinref part="U$4" gate="G$1" pin="P$1"/>
+<wire x1="182.88" y1="68.58" x2="170.18" y2="68.58" width="0.1524" layer="91"/>
+<label x="170.18" y="68.58" size="1.778" layer="95"/>
+</segment>
 </net>
 <net name="IRQ" class="0">
@@
 </segment>
 </net>
-<net name="N$2" class="0">
-<segment>
-<pinref part="U$3" gate="G$1" pin="LED2"/>
-<wire x1="104.14" y1="83.82" x2="129.54" y2="83.82" width="0.1524" layer="91"/>
-</segment>
-</net>
-<net name="N$3" class="0">
-<segment>
-<pinref part="U$3" gate="G$1" pin="LED1"/>
-<wire x1="104.14" y1="78.74" x2="129.54" y2="78.74" width="0.1524" layer="91"/>
-</segment>
-</net>
 <net name="SW" class="0">
 <segment>
 <pinref part="U$3" gate="G$1" pin="SW"/>
-<wire x1="104.14" y1="73.66" x2="129.54" y2="73.66" width="0.1524" layer="91"/>
-<label x="127" y="73.66" size="1.778" layer="95"/>
+<wire x1="104.14" y1="73.66" x2="121.92" y2="73.66" width="0.1524" layer="91"/>
+<label x="116.84" y="73.66" size="1.778" layer="95"/>
 </segment>
 </net>
@@
 <segment>
 <pinref part="U$3" gate="G$1" pin="RF-IN"/>
-<wire x1="104.14" y1="68.58" x2="129.54" y2="68.58" width="0.1524" layer="91"/>
-<label x="124.46" y="68.58" size="1.778" layer="95"/>
+<wire x1="104.14" y1="68.58" x2="121.92" y2="68.58" width="0.1524" layer="91"/>
+<label x="116.84" y="68.58" size="1.778" layer="95"/>
 </segment>
 </net>
@@
 <segment>
 <pinref part="U$3" gate="G$1" pin="ANT"/>
-<wire x1="104.14" y1="88.9" x2="129.54" y2="88.9" width="0.1524" layer="91"/>
+<wire x1="104.14" y1="88.9" x2="121.92" y2="88.9" width="0.1524" layer="91"/>
 <label x="116.84" y="88.9" size="1.778" layer="95"/>
 </segment>
 </net>
+<net name="LED2" class="0">
+<segment>
+<pinref part="U$3" gate="G$1" pin="LED2"/>
+<wire x1="104.14" y1="83.82" x2="121.92" y2="83.82" width="0.1524" layer="91"/>
+<label x="116.84" y="83.82" size="1.778" layer="95"/>
+</segment>
+<segment>
+<pinref part="U$5" gate="G$1" pin="PIN"/>
+<wire x1="182.88" y1="86.36" x2="170.18" y2="86.36" width="0.1524" layer="91"/>
+<label x="170.18" y="86.36" size="1.778" layer="95"/>
+</segment>
+</net>
+<net name="LED1" class="0">
+<segment>
+<pinref part="U$3" gate="G$1" pin="LED1"/>
+<wire x1="104.14" y1="78.74" x2="121.92" y2="78.74" width="0.1524" layer="91"/>
+<label x="116.84" y="78.74" size="1.778" layer="95"/>
+</segment>
+<segment>
+<pinref part="U$4" gate="G$1" pin="PIN"/>
+<wire x1="182.88" y1="71.12" x2="170.18" y2="71.12" width="0.1524" layer="91"/>
+<label x="170.18" y="71.12" size="1.778" layer="95"/>
+</segment>
+</net>
