File: schematics/KPNN2024/Board/RADIO.sch (EAGLE design)
At the start: 7 parts, among them J1 U.FL-R-SMT-1_10_, J2 U.FL-R-SMT-1_10_

Commit message: SUS
Parts:
- added U$6: PBS_SMD_X13, UNKNOWN-2024:PBS_SMD_X13
- added U$7: PBS_SMD_X9, UNKNOWN-2024:PBS_SMD_X9
Connections:
- new net ADC_FOTO: U$6.10
- new net CE_RADIO: U$7.1
- new net CS_RADIO: U$7.2
- new net DIR_DRIVER: U$6.1
- new net IRQ_RADIO: U$7.3
- new net LATCH_SR: U$6.5
- new net MISO_RADIO: U$7.5
- new net MISO_SR: U$6.8
- new net MOSI_RADIO: U$7.4
- new net MOSI_SR: U$6.9
- new net OE_SR: U$6.6
- new net RX1_BLE: U$6.4
- new net RX2_GPS: U$7.8
- new net SCK_RADIO: U$7.6
- new net SCK_SR: U$6.7
- new net STEP_DRIVER: U$6.2
- new net SV: U$6.11
- new net SW_WMP: U$7.9
- new net TX1_BLE: U$6.3
- new net TX2_GPS: U$7.7
- net 3V3: now also U$6.13
- net GND: now also U$6.12
Changed lines of the file:
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@@
 <part name="U$4" library="UNKNOWN-2024" deviceset="CONNECT_3" device=""/>
 <part name="U$5" library="UNKNOWN-2024" deviceset="CONNECT_3" device=""/>
+<part name="U$6" library="UNKNOWN-2024" deviceset="PBS_SMD_X13" device=""/>
+<part name="U$7" library="UNKNOWN-2024" deviceset="PBS_SMD_X9" device=""/>
 </parts>
 <sheets>
@@
 <attribute name="NAME" x="187.96" y="93.98" size="1.778" layer="94"/>
 </instance>
+<instance part="U$6" gate="G$1" x="43.18" y="116.84" smashed="yes">
+<attribute name="NAME" x="36.83" y="135.255" size="1.778" layer="95"/>
+<attribute name="VALUE" x="36.83" y="96.52" size="1.778" layer="96"/>
+</instance>
+<instance part="U$7" gate="G$1" x="88.9" y="121.92" smashed="yes">
+<attribute name="NAME" x="82.55" y="135.255" size="1.778" layer="95"/>
+<attribute name="VALUE" x="82.55" y="106.68" size="1.778" layer="96"/>
+</instance>
 </instances>
 <busses>
@@
 <label x="170.18" y="73.66" size="1.778" layer="95"/>
 </segment>
+<segment>
+<wire x1="40.64" y1="104.14" x2="10.16" y2="104.14" width="0.1524" layer="91"/>
+<pinref part="U$6" gate="G$1" pin="12"/>
+<label x="10.16" y="104.14" size="1.778" layer="95"/>
+</segment>
 </net>
 <net name="3V3" class="0">
@@
 <label x="170.18" y="68.58" size="1.778" layer="95"/>
 </segment>
+<segment>
+<pinref part="U$6" gate="G$1" pin="13"/>
+<wire x1="40.64" y1="101.6" x2="10.16" y2="101.6" width="0.1524" layer="91"/>
+<label x="10.16" y="101.6" size="1.778" layer="95"/>
+</segment>
 </net>
 <net name="IRQ" class="0">
@@
 </segment>
 </net>
+<net name="DIR_DRIVER" class="0">
+<segment>
+<pinref part="U$6" gate="G$1" pin="1"/>
+<wire x1="40.64" y1="132.08" x2="10.16" y2="132.08" width="0.1524" layer="91"/>
+<label x="10.16" y="132.08" size="1.778" layer="95"/>
+</segment>
+</net>
+<net name="STEP_DRIVER" class="0">
+<segment>
+<pinref part="U$6" gate="G$1" pin="2"/>
+<wire x1="40.64" y1="129.54" x2="10.16" y2="129.54" width="0.1524" layer="91"/>
+<label x="10.16" y="129.54" size="1.778" layer="95"/>
+</segment>
+</net>
+<net name="TX1_BLE" class="0">
+<segment>
+<pinref part="U$6" gate="G$1" pin="3"/>
+<wire x1="40.64" y1="127" x2="10.16" y2="127" width="0.1524" layer="91"/>
+<label x="10.16" y="127" size="1.778" layer="95"/>
+</segment>
+</net>
+<net name="RX1_BLE" class="0">
+<segment>
+<wire x1="40.64" y1="124.46" x2="10.16" y2="124.46" width="0.1524" layer="91"/>
+<pinref part="U$6" gate="G$1" pin="4"/>
+<label x="10.16" y="124.46" size="1.778" layer="95"/>
+</segment>
+</net>
+<net name="LATCH_SR" class="0">
+<segment>
+<wire x1="40.64" y1="121.92" x2="10.16" y2="121.92" width="0.1524" layer="91"/>
+<pinref part="U$6" gate="G$1" pin="5"/>
+<label x="10.16" y="121.92" size="1.778" layer="95"/>
+</segment>
+</net>
+<net name="OE_SR" class="0">
+<segment>
+<wire x1="40.64" y1="119.38" x2="10.16" y2="119.38" width="0.1524" layer="91"/>
+<pinref part="U$6" gate="G$1" pin="6"/>
+<label x="10.16" y="119.38" size="1.778" layer="95"/>
+</segment>
+</net>
+<net name="SCK_SR" class="0">
+<segment>
+<wire x1="40.64" y1="116.84" x2="10.16" y2="116.84" width="0.1524" layer="91"/>
+<pinref part="U$6" gate="G$1" pin="7"/>
+<label x="10.16" y="116.84" size="1.778" layer="95"/>
+</segment>
+</net>
+<net name="MISO_SR" class="0">
+<segment>
+<wire x1="40.64" y1="114.3" x2="10.16" y2="114.3" width="0.1524" layer="91"/>
+<pinref part="U$6" gate="G$1" pin="8"/>
+<label x="10.16" y="114.3" size="1.778" layer="95"/>
+</segment>
+</net>
+<net name="MOSI_SR" class="0">
+<segment>
+<wire x1="40.64" y1="111.76" x2="10.16" y2="111.76" width="0.1524" layer="91"/>
+<pinref part="U$6" gate="G$1" pin="9"/>
+<label x="10.16" y="111.76" size="1.778" layer="95"/>
+</segment>
+</net>
+<net name="ADC_FOTO" class="0">
+<segment>
+<wire x1="40.64" y1="109.22" x2="10.16" y2="109.22" width="0.1524" layer="91"/>
+<pinref part="U$6" gate="G$1" pin="10"/>
+<label x="10.16" y="109.22" size="1.778" layer="95"/>
+</segment>
+</net>
+<net name="SV" class="0">
+<segment>
+<wire x1="40.64" y1="106.68" x2="10.16" y2="106.68" width="0.1524" layer="91"/>
+<pinref part="U$6" gate="G$1" pin="11"/>
+<label x="10.16" y="106.68" size="1.778" layer="95"/>
+</segment>
+</net>
+<net name="CE_RADIO" class="0">
+<segment>
+<wire x1="86.36" y1="132.08" x2="55.88" y2="132.08" width="0.1524" layer="91"/>
+<pinref part="U$7" gate="G$1" pin="1"/>
+<label x="55.88" y="132.08" size="1.778" layer="95"/>
+</segment>
+</net>
+<net name="CS_RADIO" class="0">
+<segment>
+<wire x1="86.36" y1="129.54" x2="55.88" y2="129.54" width="0.1524" layer="91"/>
+<pinref part="U$7" gate="G$1" pin="2"/>
+<label x="55.88" y="129.54" size="1.778" layer="95"/>
+</segment>
+</net>
+<net name="IRQ_RADIO" class="0">
+<segment>
+<wire x1="86.36" y1="127" x2="55.88" y2="127" width="0.1524" layer="91"/>
+<pinref part="U$7" gate="G$1" pin="3"/>
+<label x="55.88" y="127" size="1.778" layer="95"/>
+</segment>
+</net>
+<net name="MOSI_RADIO" class="0">
+<segment>
+<wire x1="86.36" y1="124.46" x2="55.88" y2="124.46" width="0.1524" layer="91"/>
+<pinref part="U$7" gate="G$1" pin="4"/>
+<label x="55.88" y="124.46" size="1.778" layer="95"/>
+</segment>
+</net>
+<net name="MISO_RADIO" class="0">
+<segment>
+<wire x1="86.36" y1="121.92" x2="55.88" y2="121.92" width="0.1524" layer="91"/>
+<pinref part="U$7" gate="G$1" pin="5"/>
+<label x="55.88" y="121.92" size="1.778" layer="95"/>
+</segment>
+</net>
+<net name="SCK_RADIO" class="0">
+<segment>
+<wire x1="86.36" y1="119.38" x2="55.88" y2="119.38" width="0.1524" layer="91"/>
+<pinref part="U$7" gate="G$1" pin="6"/>
+<label x="55.88" y="119.38" size="1.778" layer="95"/>
+</segment>
+</net>
+<net name="TX2_GPS" class="0">
+<segment>
+<wire x1="86.36" y1="116.84" x2="55.88" y2="116.84" width="0.1524" layer="91"/>
+<pinref part="U$7" gate="G$1" pin="7"/>
+<label x="55.88" y="116.84" size="1.778" layer="95"/>
+</segment>
+</net>
+<net name="RX2_GPS" class="0">
+<segment>
+<wire x1="86.36" y1="114.3" x2="55.88" y2="114.3" width="0.1524" layer="91"/>
+<pinref part="U$7" gate="G$1" pin="8"/>
+<label x="55.88" y="114.3" size="1.778" layer="95"/>
+</segment>
+</net>
+<net name="SW_WMP" class="0">
+<segment>
+<wire x1="86.36" y1="111.76" x2="55.88" y2="111.76" width="0.1524" layer="91"/>
+<pinref part="U$7" gate="G$1" pin="9"/>
+<label x="55.88" y="111.76" size="1.778" layer="95"/>
+</segment>
+</net>

Commit message: кцуенгшщозлдх
Parts:
- added U$8: PBS_SMD_X13, UNKNOWN-2024:PBS_SMD_X13
Connections:
- removed net CE: U$2.CE
- removed net CSN: U$2.CSN
- removed net IRQ: U$2.IRQ
- removed net MISO: U$2.MISO
- removed net MOSI: U$2.MOSI
- removed net RX: U$1.RX
- removed net SCK: U$2.SCK
- removed net SV: U$6.11
- removed net SW: U$3.SW
- removed net TX: U$1.TX
- net 3V3: now also U$8.13
- net 5V: now also U$6.11, U$8.11
- net ADC_FOTO: now also U$8.10
- net CE_RADIO: now also U$2.CE
- net CS_RADIO: now also U$2.CSN
- net DIR_DRIVER: now also U$8.1
- net GND: now also U$8.12
- net IRQ_RADIO: now also U$2.IRQ
- net LATCH_SR: now also U$8.5
- net MISO_RADIO: now also U$2.MISO
- net MISO_SR: now also U$8.8
- net MOSI_RADIO: now also U$2.MOSI
- net MOSI_SR: now also U$8.9
- net OE_SR: now also U$8.6
- net RX1_BLE: now also U$8.4
- net RX2_GPS: now also U$1.RX
- net SCK_RADIO: now also U$2.SCK
- net SCK_SR: now also U$8.7
- net STEP_DRIVER: now also U$8.2
- net SW_WMP: now also U$3.SW
- net TX1_BLE: now also U$8.3
- net TX2_GPS: now also U$1.TX

Commit message: горншлщ90зд-жхэзжотрм с
Connections:
- net 3V3: now also U$8.1; no longer U$8.13
- net 5V: now also U$8.3; no longer U$8.11
- net ADC_FOTO: now also U$8.4; no longer U$8.10
- net DIR_DRIVER: now also U$8.13; no longer U$8.1
- net GND: now also U$8.2; no longer U$8.12
- net LATCH_SR: now also U$8.9; no longer U$8.5
- net MISO_SR: now also U$8.6; no longer U$8.8
- net MOSI_SR: now also U$8.5; no longer U$8.9
- net OE_SR: now also U$8.8; no longer U$8.6
- net RX1_BLE: now also U$8.10; no longer U$8.4
- net STEP_DRIVER: now also U$8.12; no longer U$8.2
- net TX1_BLE: now also U$8.11; no longer U$8.3
Other:
- moved on the sheet: U$8
Changed lines of the file:
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@@
 <attribute name="VALUE" x="82.55" y="106.68" size="1.778" layer="96"/>
 </instance>
-<instance part="U$8" gate="G$1" x="142.24" y="116.84" smashed="yes">
-<attribute name="NAME" x="135.89" y="135.255" size="1.778" layer="95"/>
-<attribute name="VALUE" x="135.89" y="96.52" size="1.778" layer="96"/>
+<instance part="U$8" gate="G$1" x="111.76" y="116.84" smashed="yes" rot="R180">
+<attribute name="NAME" x="118.11" y="98.425" size="1.778" layer="95" rot="R180"/>
+<attribute name="VALUE" x="118.11" y="137.16" size="1.778" layer="96" rot="R180"/>
 </instance>
 </instances>
@@
 </segment>
 <segment>
-<wire x1="139.7" y1="104.14" x2="109.22" y2="104.14" width="0.1524" layer="91"/>
-<pinref part="U$8" gate="G$1" pin="12"/>
-<label x="109.22" y="104.14" size="1.778" layer="95"/>
+<wire x1="144.78" y1="104.14" x2="114.3" y2="104.14" width="0.1524" layer="91"/>
+<label x="129.54" y="104.14" size="1.778" layer="95"/>
+<pinref part="U$8" gate="G$1" pin="2"/>
 </segment>
 </net>
@@
 </segment>
 <segment>
-<pinref part="U$8" gate="G$1" pin="13"/>
-<wire x1="139.7" y1="101.6" x2="109.22" y2="101.6" width="0.1524" layer="91"/>
-<label x="109.22" y="101.6" size="1.778" layer="95"/>
+<wire x1="144.78" y1="101.6" x2="114.3" y2="101.6" width="0.1524" layer="91"/>
+<label x="129.54" y="101.6" size="1.778" layer="95"/>
+<pinref part="U$8" gate="G$1" pin="1"/>
 </segment>
 </net>
@@
 </segment>
 <segment>
-<wire x1="139.7" y1="106.68" x2="109.22" y2="106.68" width="0.1524" layer="91"/>
-<pinref part="U$8" gate="G$1" pin="11"/>
-<label x="109.22" y="106.68" size="1.778" layer="95"/>
+<wire x1="144.78" y1="106.68" x2="114.3" y2="106.68" width="0.1524" layer="91"/>
+<label x="129.54" y="106.68" size="1.778" layer="95"/>
+<pinref part="U$8" gate="G$1" pin="3"/>
 </segment>
 </net>
@@
 </segment>
 <segment>
-<pinref part="U$8" gate="G$1" pin="1"/>
-<wire x1="139.7" y1="132.08" x2="109.22" y2="132.08" width="0.1524" layer="91"/>
-<label x="109.22" y="132.08" size="1.778" layer="95"/>
+<wire x1="144.78" y1="132.08" x2="114.3" y2="132.08" width="0.1524" layer="91"/>
+<label x="129.54" y="132.08" size="1.778" layer="95"/>
+<pinref part="U$8" gate="G$1" pin="13"/>
 </segment>
 </net>
@@
 </segment>
 <segment>
-<pinref part="U$8" gate="G$1" pin="2"/>
-<wire x1="139.7" y1="129.54" x2="109.22" y2="129.54" width="0.1524" layer="91"/>
-<label x="109.22" y="129.54" size="1.778" layer="95"/>
+<wire x1="144.78" y1="129.54" x2="114.3" y2="129.54" width="0.1524" layer="91"/>
+<label x="129.54" y="129.54" size="1.778" layer="95"/>
+<pinref part="U$8" gate="G$1" pin="12"/>
 </segment>
 </net>
@@
 </segment>
 <segment>
-<pinref part="U$8" gate="G$1" pin="3"/>
-<wire x1="139.7" y1="127" x2="109.22" y2="127" width="0.1524" layer="91"/>
-<label x="109.22" y="127" size="1.778" layer="95"/>
+<wire x1="144.78" y1="127" x2="114.3" y2="127" width="0.1524" layer="91"/>
+<label x="129.54" y="127" size="1.778" layer="95"/>
+<pinref part="U$8" gate="G$1" pin="11"/>
 </segment>
 </net>
@@
 </segment>
 <segment>
-<wire x1="139.7" y1="124.46" x2="109.22" y2="124.46" width="0.1524" layer="91"/>
-<pinref part="U$8" gate="G$1" pin="4"/>
-<label x="109.22" y="124.46" size="1.778" layer="95"/>
+<wire x1="144.78" y1="124.46" x2="114.3" y2="124.46" width="0.1524" layer="91"/>
+<label x="129.54" y="124.46" size="1.778" layer="95"/>
+<pinref part="U$8" gate="G$1" pin="10"/>
 </segment>
 </net>
@@
 </segment>
 <segment>
-<wire x1="139.7" y1="121.92" x2="109.22" y2="121.92" width="0.1524" layer="91"/>
-<pinref part="U$8" gate="G$1" pin="5"/>
-<label x="109.22" y="121.92" size="1.778" layer="95"/>
+<wire x1="144.78" y1="121.92" x2="114.3" y2="121.92" width="0.1524" layer="91"/>
+<label x="129.54" y="121.92" size="1.778" layer="95"/>
+<pinref part="U$8" gate="G$1" pin="9"/>
 </segment>
 </net>
@@
 </segment>
 <segment>
-<wire x1="139.7" y1="119.38" x2="109.22" y2="119.38" width="0.1524" layer="91"/>
-<pinref part="U$8" gate="G$1" pin="6"/>
-<label x="109.22" y="119.38" size="1.778" layer="95"/>
+<wire x1="144.78" y1="119.38" x2="114.3" y2="119.38" width="0.1524" layer="91"/>
+<label x="129.54" y="119.38" size="1.778" layer="95"/>
+<pinref part="U$8" gate="G$1" pin="8"/>
 </segment>
 </net>
@@
 </segment>
 <segment>
-<wire x1="139.7" y1="116.84" x2="109.22" y2="116.84" width="0.1524" layer="91"/>
+<wire x1="144.78" y1="116.84" x2="114.3" y2="116.84" width="0.1524" layer="91"/>
+<label x="129.54" y="116.84" size="1.778" layer="95"/>
 <pinref part="U$8" gate="G$1" pin="7"/>
-<label x="109.22" y="116.84" size="1.778" layer="95"/>
 </segment>
 </net>
@@
 </segment>
 <segment>
-<wire x1="139.7" y1="114.3" x2="109.22" y2="114.3" width="0.1524" layer="91"/>
-<pinref part="U$8" gate="G$1" pin="8"/>
-<label x="109.22" y="114.3" size="1.778" layer="95"/>
+<wire x1="144.78" y1="114.3" x2="114.3" y2="114.3" width="0.1524" layer="91"/>
+<label x="129.54" y="114.3" size="1.778" layer="95"/>
+<pinref part="U$8" gate="G$1" pin="6"/>
 </segment>
 </net>
@@
 </segment>
 <segment>
-<wire x1="139.7" y1="111.76" x2="109.22" y2="111.76" width="0.1524" layer="91"/>
-<pinref part="U$8" gate="G$1" pin="9"/>
-<label x="109.22" y="111.76" size="1.778" layer="95"/>
+<wire x1="144.78" y1="111.76" x2="114.3" y2="111.76" width="0.1524" layer="91"/>
+<label x="129.54" y="111.76" size="1.778" layer="95"/>
+<pinref part="U$8" gate="G$1" pin="5"/>
 </segment>
 </net>
@@
 </segment>
 <segment>
-<wire x1="139.7" y1="109.22" x2="109.22" y2="109.22" width="0.1524" layer="91"/>
-<pinref part="U$8" gate="G$1" pin="10"/>
-<label x="109.22" y="109.22" size="1.778" layer="95"/>
-</segment>
-</net>
+<wire x1="144.78" y1="109.22" x2="114.3" y2="109.22" width="0.1524" layer="91"/>
+<label x="129.54" y="109.22" size="1.778" layer="95"/>
+<pinref part="U$8" gate="G$1" pin="4"/>
+</segment>
+</net>

Commit message: плата рпарпарпараарпарпарпааарпарпарпауекуекуекусруркра
Parts:
- added LED1, LED2: (no value), led:LEDCHIPLED_0603
- added R1, R2: (no value), rcl:R-US_R0603
Connections:
- removed net LED1: U$3.LED1, U$4.PIN
- removed net LED2: U$3.LED2, U$5.PIN
- new net N$1: LED1.C, R1.2
- new net N$2: LED2.C, R2.2
- new net N$3: LED1.A, U$4.PIN
- new net N$4: LED2.A, U$5.PIN
- new net N$5: R2.1, U$3.LED2
- new net N$6: R1.1, U$3.LED1
Changed lines of the file:
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@@
 <part name="U$7" library="UNKNOWN-2024" deviceset="PBS_SMD_X9" device=""/>
 <part name="U$8" library="UNKNOWN-2024" deviceset="PBS_SMD_X13" device=""/>
+<part name="LED1" library="led" library_urn="urn:adsk.eagle:library:259" deviceset="LED" device="CHIPLED_0603" package3d_urn="urn:adsk.eagle:package:15822/2"/>
+<part name="LED2" library="led" library_urn="urn:adsk.eagle:library:259" deviceset="LED" device="CHIPLED_0603" package3d_urn="urn:adsk.eagle:package:15822/2"/>
+<part name="R1" library="rcl" library_urn="urn:adsk.eagle:library:334" deviceset="R-US_" device="R0603" package3d_urn="urn:adsk.eagle:package:23555/3"/>
+<part name="R2" library="rcl" library_urn="urn:adsk.eagle:library:334" deviceset="R-US_" device="R0603" package3d_urn="urn:adsk.eagle:package:23555/3"/>
 </parts>
 <sheets>
@@
 <attribute name="VALUE" x="118.11" y="137.16" size="1.778" layer="96" rot="R180"/>
 </instance>
+<instance part="LED1" gate="G$1" x="162.56" y="71.12" smashed="yes" rot="R270">
+<attribute name="NAME" x="157.988" y="67.564" size="1.778" layer="95"/>
+<attribute name="VALUE" x="157.988" y="65.405" size="1.778" layer="96"/>
+</instance>
+<instance part="LED2" gate="G$1" x="162.56" y="86.36" smashed="yes" rot="R270">
+<attribute name="NAME" x="157.988" y="82.804" size="1.778" layer="95"/>
+<attribute name="VALUE" x="157.988" y="80.645" size="1.778" layer="96"/>
+</instance>
+<instance part="R1" gate="G$1" x="147.32" y="71.12" smashed="yes">
+<attribute name="NAME" x="143.51" y="72.6186" size="1.778" layer="95"/>
+<attribute name="VALUE" x="143.51" y="67.818" size="1.778" layer="96"/>
+</instance>
+<instance part="R2" gate="G$1" x="147.32" y="86.36" smashed="yes">
+<attribute name="VALUE" x="143.51" y="83.058" size="1.778" layer="96"/>
+</instance>
 </instances>
 <busses>
@@
 </segment>
 </net>
-<net name="LED2" class="0">
-<segment>
-<pinref part="U$3" gate="G$1" pin="LED2"/>
-<wire x1="104.14" y1="83.82" x2="121.92" y2="83.82" width="0.1524" layer="91"/>
-<label x="116.84" y="83.82" size="1.778" layer="95"/>
-</segment>
-<segment>
-<pinref part="U$5" gate="G$1" pin="PIN"/>
-<wire x1="182.88" y1="86.36" x2="170.18" y2="86.36" width="0.1524" layer="91"/>
-<label x="170.18" y="86.36" size="1.778" layer="95"/>
-</segment>
-</net>
-<net name="LED1" class="0">
-<segment>
-<pinref part="U$3" gate="G$1" pin="LED1"/>
-<wire x1="104.14" y1="78.74" x2="121.92" y2="78.74" width="0.1524" layer="91"/>
-<label x="116.84" y="78.74" size="1.778" layer="95"/>
-</segment>
-<segment>
-<pinref part="U$4" gate="G$1" pin="PIN"/>
-<wire x1="182.88" y1="71.12" x2="170.18" y2="71.12" width="0.1524" layer="91"/>
-<label x="170.18" y="71.12" size="1.778" layer="95"/>
-</segment>
-</net>
 <net name="DIR_DRIVER" class="0">
 <segment>
@@
 <wire x1="104.14" y1="73.66" x2="121.92" y2="73.66" width="0.1524" layer="91"/>
 <label x="116.84" y="73.66" size="1.778" layer="95"/>
+</segment>
+</net>
+<net name="N$1" class="0">
+<segment>
+<pinref part="LED1" gate="G$1" pin="C"/>
+<pinref part="R1" gate="G$1" pin="2"/>
+<wire x1="152.4" y1="71.12" x2="157.48" y2="71.12" width="0.1524" layer="91"/>
+</segment>
+</net>
+<net name="N$2" class="0">
+<segment>
+<pinref part="LED2" gate="G$1" pin="C"/>
+<pinref part="R2" gate="G$1" pin="2"/>
+<wire x1="152.4" y1="86.36" x2="157.48" y2="86.36" width="0.1524" layer="91"/>
+</segment>
+</net>
+<net name="N$3" class="0">
+<segment>
+<pinref part="U$4" gate="G$1" pin="PIN"/>
+<pinref part="LED1" gate="G$1" pin="A"/>
+<wire x1="165.1" y1="71.12" x2="182.88" y2="71.12" width="0.1524" layer="91"/>
+</segment>
+</net>
+<net name="N$4" class="0">
+<segment>
+<pinref part="U$5" gate="G$1" pin="PIN"/>
+<pinref part="LED2" gate="G$1" pin="A"/>
+<wire x1="165.1" y1="86.36" x2="182.88" y2="86.36" width="0.1524" layer="91"/>
+</segment>
+</net>
+<net name="N$5" class="0">
+<segment>
+<pinref part="U$3" gate="G$1" pin="LED2"/>
+<pinref part="R2" gate="G$1" pin="1"/>
+<wire x1="104.14" y1="83.82" x2="142.24" y2="83.82" width="0.1524" layer="91"/>
+<wire x1="142.24" y1="83.82" x2="142.24" y2="86.36" width="0.1524" layer="91"/>
+</segment>
+</net>
+<net name="N$6" class="0">
+<segment>
+<pinref part="U$3" gate="G$1" pin="LED1"/>
+<pinref part="R1" gate="G$1" pin="1"/>
+<wire x1="104.14" y1="78.74" x2="142.24" y2="78.74" width="0.1524" layer="91"/>
+<wire x1="142.24" y1="78.74" x2="142.24" y2="71.12" width="0.1524" layer="91"/>
 </segment>
 </net>
@@
 </schematic>
 </drawing>
+<compatibility>
+<note version="8.2" severity="warning">
+Since Version 8.2, EAGLE supports online libraries. The ids
+of those online libraries will not be understood (or retained)
+with this version.
+</note>
+<note version="8.3" severity="warning">
+Since Version 8.3, EAGLE supports URNs for individual library
+assets (packages, symbols, and devices). The URNs of those assets
+will not be understood (or retained) with this version.
+</note>
+<note version="8.3" severity="warning">
+Since Version 8.3, EAGLE supports the association of 3D packages
+with devices in libraries, schematics, and board files. Those 3D
+packages will not be understood (or retained) with this version.
+</note>
+<note version="8.4" severity="warning">
+Since Version 8.4, EAGLE supports properties for SPICE simulation.
+Probes in schematics and SPICE mapping objects found in parts and library devices
+will not be understood with this version. Update EAGLE to the latest version
+for full support of SPICE simulation.
+</note>
+</compatibility>
 </eagle>
