File: schematics/KPNN2024/Board/MK.brd (EAGLE design)
At the start: 68.9 x 68.9 mm, 12 parts

Commit message: плата МК под разводку
Parts:
- removed U$1: PBS_SMD_X13, UNKNOWN-2024:PBD_SMD_X13
- removed U$3: PBS_SMD_X9, UNKNOWN-2024:PBS_SMD_X9
- added U$4: PBS_SMD_X13, UNKNOWN-2024:PBD_SMD_X13
- added U$6: PBS_SMD_X9, UNKNOWN-2024:PBS_SMD_X9
- BME280: value BME280 -> BME280BME280-PINS-ONLY; device UNKNOWN-2024:BME280 -> UNKNOWN-2024:BME280-PINS-ONLY
- moved BME280 35.0 mm to (93.8, 52.8)
- moved BUZZER 14.2 mm to (91.6, 30.2)
- moved R9 14.2 mm to (91.8, 31.2)
- moved R10 14.2 mm to (91.8, 33.6)
- moved U$20 14.2 mm to (91.8, 28.3)
- moved U$5 10.6 mm to (49.4, 41.6), turned to 90 degrees
Connections:
- removed net D0: MICRO_SD.DAT0
- net 3V3: now also BME280.P$4, U$4.1; no longer BME280.P$1, U$1.13
- net 5V: now also U$4.3; no longer U$1.11
- net ADC_FOTO: now also U$4.4; no longer U$1.10
- net CE_RADIO: now also U$6.9; no longer U$3.1
- net CS_RADIO: now also U$6.8; no longer U$3.2
- net D0_SD: now also MICRO_SD.DAT0
- net DIR_DRIVER: now also U$4.13; no longer U$1.1
- net GND: now also BME280.P$3, U$4.2; no longer BME280.P$2, U$1.12
- net IRQ_RADIO: now also U$6.7; no longer U$3.3
- net LATCH_SR: now also U$4.9, U$5.23; no longer U$1.5, U$5.21
- net MISO_RADIO: now also U$6.5; no longer U$3.5
- net MISO_SR: now also U$4.6; no longer U$1.8
- net MOSI_RADIO: now also U$6.6; no longer U$3.4
- net MOSI_SR: now also U$4.5; no longer U$1.9
- net OE_SR: now also U$4.8, U$5.25; no longer U$1.6, U$5.23
- net RX1_BLE: now also U$4.10; no longer U$1.4
- net RX2_GPS: now also U$6.2; no longer U$3.8
- net SCK_RADIO: now also U$6.4; no longer U$3.6
- net SCK_SR: now also U$4.7; no longer U$1.7
- net SCL: now also BME280.P$2; no longer BME280.P$3
- net SDA: now also BME280.P$1; no longer BME280.P$4
- net STEP_DRIVER: now also U$4.12; no longer U$1.2
- net SWITCH: now also U$5.21; no longer U$5.15
- net SW_AMP: now also U$6.1; no longer U$3.9
- net TX1_BLE: now also U$4.11; no longer U$1.3
- net TX2_GPS: now also U$6.3; no longer U$3.7
