File: schematics/KPNN2024/Board/MK.brd (EAGLE design)
At the start: 68.9 x 68.9 mm, 12 parts

Commit message: `1234567890000-=qwertyuiop[]asdfghjkl;'zxcvbnm,./
Parts:
- moved BME280 65.2 mm to (28.6, 53.4)
- moved BUZZER 63.4 mm to (29.0, 40.0)
- moved R10 63.4 mm to (29.2, 43.4)
- moved R9 63.4 mm to (29.2, 41.0)
- moved U$20 63.4 mm to (29.2, 38.1)
Routing:
- net 3V3: track 0.00 -> 140.7 mm, vias 0 -> 3
- net GND: track 0.00 -> 131.5 mm, vias 0 -> 4
- net MISO_RADIO: track 0.00 -> 101.8 mm, vias 0 -> 3
- net 5V: track 0.00 -> 89.8 mm, vias 0 -> 2
- net SCK_RADIO: track 0.00 -> 80.8 mm
- net D0_SD: track 0.00 -> 76.0 mm, vias 0 -> 1
- net SCK_SR: track 0.00 -> 73.8 mm, vias 0 -> 2
- net ADC_FOTO: track 0.00 -> 58.7 mm, vias 0 -> 2
- net SD_CK: track 0.00 -> 52.2 mm, vias 0 -> 1
- net SDA: track 0.00 -> 45.5 mm, vias 0 -> 1
- net SCL: track 0.00 -> 44.9 mm, vias 0 -> 1
- net MOSI_RADIO: track 0.00 -> 27.3 mm
- net RX2_GPS: track 0.00 -> 26.1 mm
- net CS_RADIO: track 0.00 -> 25.3 mm
- net SW_AMP: track 0.00 -> 24.6 mm
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
Commit message: sdfghgfds
Parts:
- added C1: (no value), rcl:C0603
- added R3, R4: 5k1, rcl:R0603
- added R5, R6: 10k, rcl:R0603
- moved R9 0.28 mm to (29.0, 41.2)
Connections:
- net 3V3: now also C1.2, R3.2, R4.2, R5.1, R6.1
- net CMD_SD: now also R6.2
- net D0_SD: now also R5.2
- net GND: now also C1.1
- net SCL: now also R4.1
- net SDA: now also R3.1
Routing:
- net 3V3: track 140.7 -> 159.0 mm, vias 3 -> 5
- net SDA: track 45.5 -> 54.3 mm
- net D0_SD: track 76.0 -> 81.6 mm
- net SCL: track 44.9 -> 49.3 mm
- net GND: track 131.5 -> 133.0 mm
- net CMD_SD: track 24.3 -> 24.9 mm

Commit message: когда фондю?
Parts:
- moved BUZZER 0.40 mm to (29.0, 39.6), flipped to the top, turned to 0 degrees
- moved MICRO_SD 0.10 mm to (16.3, 9.45)
Routing:
- net 3V3: track 159.0 -> 180.9 mm, vias 5 -> 4
- net GND: track 133.0 -> 140.7 mm, vias 4 -> 5
- net SCL: track 49.3 -> 47.4 mm
- net 5V: track 89.8 -> 89.4 mm, vias 2 -> 1
- net MISO_RADIO: track 101.8 -> 101.9 mm, vias 3 -> 1
- added copper zone on layer 1, net GND
- added copper zone on layer 16, net GND

Commit message: добавлены стл корпусных деталей
Parts:
- C1: value (none) -> 100nF
Changed lines of the file:
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@@
 <attribute name="VALUE" x="28.396053125" y="30.298025" size="1.27" layer="27" rot="R135"/>
 </element>
-<element name="C1" library="rcl" library_urn="urn:adsk.eagle:library:334" package="C0603" package3d_urn="urn:adsk.eagle:package:23616/2" value="" x="26.2" y="26.6" smashed="yes" rot="R135">
+<element name="C1" library="rcl" library_urn="urn:adsk.eagle:library:334" package="C0603" package3d_urn="urn:adsk.eagle:package:23616/2" value="100nF" x="26.2" y="26.6" smashed="yes" rot="R135">
 <attribute name="NAME" x="22.8" y="29.298028125" size="1.27" layer="25" rot="R315"/>
 <attribute name="POPULARITY" value="73" x="26.2" y="26.6" size="1.778" layer="27" rot="R135" display="off"/>
@@
 </polygon>
 <polygon width="0.3" layer="1">
-<vertex x="5.9" y="82.1"/>
-<vertex x="78.6" y="82.1"/>
-<vertex x="78.6" y="1.5"/>
-<vertex x="4" y="1.5"/>
-<vertex x="3.4" y="2.1"/>
-<vertex x="3.4" y="81.8"/>
-<vertex x="3.6" y="82"/>
-<vertex x="5.8" y="82"/>
+<vertex x="4.7" y="56.1"/>
+<vertex x="24.9" y="76.3"/>
+<vertex x="56.8" y="76.3"/>
+<vertex x="77.1" y="56"/>
+<vertex x="77.1" y="16.9"/>
+<vertex x="64.5" y="4.3"/>
+<vertex x="18.2" y="4.3"/>
+<vertex x="4.7" y="17.8"/>
 </polygon>
 </signal>

Commit message: ывавп лыл
Parts:
- renumbered U$20 to SI2302CDS, U$5 to STM
Routing:
- net 3V3: track 180.9 -> 177.4 mm

Commit message: Разведена плата питания
Parts:
- moved R2 1.48 mm to (69.7, 18.7)
- moved U$2 1.14 mm to (65.9, 13.9)
- moved R1 0.94 mm to (60.2, 9.50)
- moved C1 0.64 mm to (26.7, 26.2)
- moved R5 0.57 mm to (29.2, 26.8)
- moved MICRO_SD 0.54 mm to (16.8, 9.65), turned to 131 degrees
- moved R6 0.50 mm to (27.0, 29.1)
Routing:
- net GND: track 140.7 -> 139.1 mm
- net 3V3: track 177.4 -> 175.8 mm
- net SWITCH: track 11.7 -> 10.5 mm
- net CMD_SD: track 24.8 -> 23.6 mm

Commit message: Платы вроде готовы
Parts:
- added STATE: (no value), led:CHIPLED_0603
- R1, R2: value 10k -> 2k
- moved R10 11.8 mm to (18.0, 39.7), flipped to the top
- moved SI2302CDS 11.7 mm to (18.0, 34.4), flipped to the top
- moved R9 11.4 mm to (18.2, 37.5), flipped to the top
- moved R1 2.13 mm to (58.6, 10.9), turned to 135 degrees
- moved U$2 2.13 mm to (64.3, 15.3)
- moved R2 2.08 mm to (68.0, 19.9)
- moved BUZZER 0.85 mm to (28.7, 38.8), turned to 90 degrees
- turned C1 to 131 degrees
- turned R5 to 311 degrees
- turned R6 to 131 degrees
Connections:
- net 3V3: no longer BME280.P$4
- net 5V: now also BME280.P$4; no longer STM.20, STM.38
- net DIR_DRIVER: now also STM.27, U$4.12; no longer STM.26, U$4.13
- net GND: now also STATE.C
- net STEP_DRIVER: now also STM.26, U$4.13; no longer STM.27, U$4.12
- net SWITCH: now also STATE.A
Routing:
- net SCK_SR: track 73.8 -> 23.9 mm
- net GND: track 139.1 -> 171.4 mm
- net ADC_FOTO: track 58.7 -> 26.5 mm
- net 5V: track 89.4 -> 62.5 mm, vias 1 -> 0
- net 3V3: track 175.8 -> 153.4 mm, vias 4 -> 2
- net BUZZER: track 20.3 -> 30.8 mm, vias 0 -> 1
- net SWITCH: track 10.5 -> 17.7 mm
- net N$13: track 6.20 -> 11.2 mm
- net STEP_DRIVER: track 11.4 -> 8.75 mm
- net DIR_DRIVER: track 8.75 -> 11.4 mm
Other:
- board text added: "3V3"
- board text added: "5V"
- board text added: "CE"
- board text added: "CS"
- board text added: "DIR"
- board text added: "FOTO"
- board text added: "GND"
- board text added: "IRQ"
- board text added: "LATCH"
- board text added: "MISO"
- board text added: "MOSI"
- board text added: "OE"
- board text added: "RX1"
- board text added: "RX2"
- board text added: "SCK"
- board text added: "STEP"
- board text added: "SW"
- board text added: "TX1"
- board text added: "TX2"

Commit message: сдклвл платы а мботрен зз
Changed lines of the file:
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@@
 <?xml version="1.0" encoding="utf-8"?>
 <!DOCTYPE eagle SYSTEM "eagle.dtd">
-<eagle version="9.4.2">
+<eagle version="9.6.2">
 <drawing>
 <settings>
-<setting alwaysvectorfont="yes"/>
+<setting alwaysvectorfont="no"/>
 <setting verticaltext="up"/>
 </settings>
@@
 </autorouter>
 <elements>
-<element name="MICRO_SD" library="UNKNOWN-2024" package="SD" value="SD" x="16.7814875" y="9.654290625" smashed="yes" rot="R131">
-<attribute name="NAME" x="16.42138125" y="14.641296875" size="1" layer="25" font="vector" ratio="15" rot="R131"/>
+<element name="MICRO_SD" library="UNKNOWN-2024" package="SD" value="SD" x="16.78" y="9.65" smashed="yes" rot="R131">
+<attribute name="NAME" x="16.419890625" y="14.637003125" size="1" layer="25" font="vector" ratio="15" rot="R131"/>
 </element>
 <element name="BUZZER" library="CanCubeSat" package="BUZZER-S8R12" value="BUZZERS8R6" x="28.7" y="38.8" smashed="yes" rot="R90">
@@
 <attribute name="VALUE" x="20.065" y="39.295" size="1" layer="27" font="vector" ratio="15"/>
 </element>
-<element name="U$2" library="UNKNOWN-2024" package="SWITCH_MSS" value="SWITCH_MSS" x="64.303021875" y="15.257525" smashed="yes" rot="R223">
-<attribute name="VALUE" x="64.924134375" y="20.4779875" size="1" layer="27" font="vector" ratio="15" rot="R223"/>
+<element name="U$2" library="UNKNOWN-2024" package="SWITCH_MSS" value="SWITCH_MSS" x="64.3" y="15.257525" smashed="yes" rot="R223">
+<attribute name="VALUE" x="64.9211125" y="20.4779875" size="1" layer="27" font="vector" ratio="15" rot="R223"/>
 </element>
 <element name="R1" library="rcl" library_urn="urn:adsk.eagle:library:334" package="R0603" package3d_urn="urn:adsk.eagle:package:23555/3" value="2k" x="58.6" y="10.9" smashed="yes" rot="R135">
@@
 <wire x1="17.0876875" y1="37.4123125" x2="17" y2="37.5" width="0.5" layer="1"/>
 <wire x1="23.6" y1="21.8" x2="23.6" y2="21.82985" width="0.5" layer="1"/>
-<wire x1="25.468565625" y1="23.698415625" x2="23.6" y2="21.82985" width="0.5" layer="1"/>
+<wire x1="25.467078125" y1="23.694125" x2="23.6" y2="21.82985" width="0.5" layer="1"/>
 <via x="23.6" y="21.8" extent="1-16" drill="0.35"/>
 <polygon width="0.3" layer="16">
@@
 <vertex x="4.7" y="17.8"/>
 </polygon>
-<wire x1="25.468565625" y1="23.698415625" x2="25.468565625" y2="23.76648125" width="0.5" layer="1"/>
+<wire x1="25.467078125" y1="23.694125" x2="25.468565625" y2="23.76648125" width="0.5" layer="1"/>
 <wire x1="25.468565625" y1="23.76648125" x2="27.25765" y2="25.55849375" width="0.5" layer="1"/>
 <wire x1="56.9" y1="63.19" x2="58.91" y2="63.19" width="0.5" layer="16"/>
@@
 <wire x1="28.642346875" y1="27.441503125" x2="30.198909375" y2="29" width="0.5" layer="1"/>
 <wire x1="30.198909375" y1="29" x2="33.1" y2="29" width="0.5" layer="1"/>
-<wire x1="24.0252375" y1="25.358778125" x2="24.2252375" y2="25.358778125" width="0.5" layer="1"/>
+<wire x1="24.02375" y1="25.3544875" x2="24.2252375" y2="25.358778125" width="0.5" layer="1"/>
 <wire x1="28.59895625" y1="27.501040625" x2="28.642346875" y2="27.441503125" width="0.5" layer="1"/>
 <wire x1="24.2252375" y1="25.358778125" x2="25.7079625" y2="26.841503125" width="0.5" layer="1"/>
@@
 <wire x1="34.487915625" y1="37.79" x2="41.9" y2="37.79" width="0.3" layer="1"/>
 <wire x1="26.442346875" y1="29.741503125" x2="34.487915625" y2="37.79" width="0.3" layer="1"/>
-<wire x1="23.303571875" y1="26.188959375" x2="26.39895625" y2="29.28434375" width="0.3" layer="1"/>
+<wire x1="23.302084375" y1="26.18466875" x2="26.39895625" y2="29.28434375" width="0.3" layer="1"/>
 <wire x1="26.39895625" y1="29.28434375" x2="26.442346875" y2="29.741503125" width="0.3" layer="1"/>
 </signal>
@@
 <contactref element="MICRO_SD" pad="CLK"/>
 <contactref element="STM" pad="24"/>
-<wire x1="24.746903125" y1="24.528596875" x2="24.431915625" y2="24.213609375" width="0.3" layer="1"/>
+<wire x1="24.745415625" y1="24.52430625" x2="24.431915625" y2="24.213609375" width="0.3" layer="1"/>
 <wire x1="24.431915625" y1="24.213609375" x2="21.9" y2="21.9923625" width="0.3" layer="1"/>
 <wire x1="21.9" y1="21.9923625" x2="21.9" y2="18" width="0.3" layer="1"/>
@@
 <contactref element="STM" pad="35"/>
 <contactref element="MICRO_SD" pad="DAT0"/>
-<wire x1="26.19023125" y1="22.8682375" x2="26.12951875" y2="22.807525" width="0.3" layer="1"/>
+<wire x1="26.18874375" y1="22.863946875" x2="26.12951875" y2="22.807525" width="0.3" layer="1"/>
 <wire x1="26.12951875" y1="22.807525" x2="22.8" y2="19.824575" width="0.3" layer="1"/>
 <wire x1="22.8" y1="19.824575" x2="22.8" y2="18.3071125" width="0.3" layer="1"/>
@@
 <contactref element="R5" pad="2"/>
 <wire x1="29.75765" y1="26.15849375" x2="29.52099375" y2="26.199" width="0.3" layer="1"/>
-<wire x1="29.52099375" y1="26.199" x2="26.19023125" y2="22.8682375" width="0.3" layer="1"/>
+<wire x1="29.52099375" y1="26.199" x2="26.18874375" y2="22.863946875" width="0.3" layer="1"/>
 </signal>
 <signal name="SWITCH">
@@
 <contactref element="STM" pad="21"/>
 <contactref element="STATE" pad="A"/>
-<wire x1="64.303021875" y1="15.257525" x2="65.260546875" y2="14.3" width="0.3" layer="1"/>
+<wire x1="64.3" y1="15.257525" x2="65.260546875" y2="14.3" width="0.3" layer="1"/>
 <wire x1="65.260546875" y1="14.3" x2="66.8" y2="14.3" width="0.3" layer="1"/>
 <wire x1="71.06065625" y1="17.7" x2="71.630328125" y2="17.130328125" width="0.3" layer="1"/>
 <wire x1="66.8" y1="14.3" x2="70.2" y2="17.7" width="0.3" layer="1"/>
 <wire x1="70.2" y1="17.7" x2="71.06065625" y2="17.7" width="0.3" layer="1"/>
-<wire x1="64.303021875" y1="15.257525" x2="62.090546875" y2="17.47" width="0.3" layer="1"/>
+<wire x1="64.3" y1="15.257525" x2="62.090546875" y2="17.47" width="0.3" layer="1"/>
 <wire x1="62.090546875" y1="17.47" x2="56.9" y2="17.47" width="0.3" layer="1"/>
 </signal>
@@
 <contactref element="R1" pad="1"/>
 <contactref element="U$2" pad="3"/>
-<wire x1="62.44538125" y1="13.525246875" x2="62.4270875" y2="13.525246875" width="0.3" layer="1"/>
+<wire x1="62.442359375" y1="13.525246875" x2="62.4270875" y2="13.525246875" width="0.3" layer="1"/>
 <wire x1="62.4270875" y1="13.525246875" x2="59.201040625" y2="10.29895625" width="0.3" layer="1"/>
 </signal>
@@
 <contactref element="R2" pad="1"/>
 <contactref element="U$2" pad="1"/>
-<wire x1="66.160659375" y1="16.9898" x2="66.2917" y2="16.9898" width="0.3" layer="1"/>
+<wire x1="66.1576375" y1="16.9898" x2="66.2917" y2="16.9898" width="0.3" layer="1"/>
 <wire x1="68.590459375" y1="19.288559375" x2="66.2917" y2="16.9898" width="0.3" layer="1"/>
 </signal>
