File: schematics/KPNN2024/Board/MK.sch (EAGLE design)
At the start: 10 parts

Commit message: Вабба Лабба Даб Даб
Connections:
- net ADC0 renamed ADC_FOTO
- removed net SCL1: U$1.PB6
- removed net SDA_BME: U$1.PB9
- net SCL: now also U$1.PB6
- net SDA: now also U$1.PB9

Commit message: я тоже
Connections:
- new net RX2_UART: U$1.PA3
- new net TX2_UART: U$1.PA2
- net SWITCH: now also U$2.P
Changed lines of the file:
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@@
 <label x="5.08" y="71.12" size="1.778" layer="95"/>
+</segment>
+<segment>
+<wire x1="304.8" y1="38.1" x2="342.9" y2="38.1" width="0.1524" layer="91"/>
+<label x="340.36" y="38.1" size="1.778" layer="95"/>
 </segment>
 </net>
@@
 <label x="5.08" y="55.88" size="1.778" layer="95"/>
 </segment>
+<segment>
+<wire x1="304.8" y1="43.18" x2="342.9" y2="43.18" width="0.1524" layer="91"/>
+<label x="340.36" y="43.18" size="1.778" layer="95"/>
+</segment>
 </net>
 <net name="CMD" class="0">
@@
 <label x="0" y="50.8" size="1.778" layer="95"/>
 </segment>
+<segment>
+<wire x1="304.8" y1="12.7" x2="342.9" y2="12.7" width="0.1524" layer="91"/>
+<label x="340.36" y="12.7" size="1.778" layer="95"/>
+</segment>
 </net>
 <net name="LATCH_SR" class="0">
@@
 <label x="0" y="91.44" size="1.778" layer="95"/>
 </segment>
+<segment>
+<wire x1="304.8" y1="17.78" x2="342.9" y2="17.78" width="0.1524" layer="91"/>
+<label x="340.36" y="17.78" size="1.778" layer="95"/>
+</segment>
 </net>
 <net name="MOSI_SR" class="0">
@@
 <label x="73.66" y="60.96" size="1.778" layer="95"/>
 </segment>
+<segment>
+<wire x1="304.8" y1="33.02" x2="342.9" y2="33.02" width="0.1524" layer="91"/>
+<label x="340.36" y="33.02" size="1.778" layer="95"/>
+</segment>
 </net>
 <net name="SCK_SR" class="0">
@@
 <label x="73.66" y="71.12" size="1.778" layer="95"/>
 </segment>
+<segment>
+<wire x1="304.8" y1="27.94" x2="342.9" y2="27.94" width="0.1524" layer="91"/>
+<label x="340.36" y="27.94" size="1.778" layer="95"/>
+</segment>
 </net>
 <net name="MOSI_RADIO" class="0">
@@
 <label x="0" y="81.28" size="1.778" layer="95"/>
 </segment>
+<segment>
+<wire x1="304.8" y1="22.86" x2="342.9" y2="22.86" width="0.1524" layer="91"/>
+<label x="340.36" y="22.86" size="1.778" layer="95"/>
+</segment>
 </net>
 <net name="RX_UART" class="0">
@@
 </segment>
 </net>
-<net name="SDA_BME" class="0">
-<segment>
-<wire x1="304.8" y1="43.18" x2="342.9" y2="43.18" width="0.1524" layer="91"/>
-<label x="340.36" y="43.18" size="1.778" layer="95"/>
-</segment>
-</net>
 <net name="D0_SD" class="0">
 <segment>
@@
 <label x="0" y="96.52" size="1.778" layer="95"/>
 </segment>
+<segment>
+<pinref part="U$2" gate="G$1" pin="P"/>
+<wire x1="149.86" y1="58.42" x2="170.18" y2="58.42" width="0.1524" layer="91"/>
+<label x="162.56" y="58.42" size="1.778" layer="95"/>
+</segment>
 </net>
 <net name="N$1" class="0">
@@
 </segment>
 </net>
-<net name="N$7" class="0">
-<segment>
-<wire x1="304.8" y1="38.1" x2="342.9" y2="38.1" width="0.1524" layer="91"/>
-</segment>
-</net>
-<net name="N$8" class="0">
-<segment>
-<wire x1="304.8" y1="33.02" x2="342.9" y2="33.02" width="0.1524" layer="91"/>
-</segment>
-</net>
-<net name="N$9" class="0">
-<segment>
-<wire x1="304.8" y1="27.94" x2="342.9" y2="27.94" width="0.1524" layer="91"/>
-</segment>
-</net>
-<net name="N$11" class="0">
-<segment>
-<wire x1="304.8" y1="22.86" x2="342.9" y2="22.86" width="0.1524" layer="91"/>
-</segment>
-</net>
+<net name="TX2_UART" class="0">
+<segment>
+<pinref part="U$1" gate="G$1" pin="PA2"/>
+<wire x1="60.96" y1="86.36" x2="83.82" y2="86.36" width="0.1524" layer="91"/>
+<label x="81.28" y="86.36" size="1.778" layer="95"/>
+</segment>
+<segment>
+<wire x1="304.8" y1="7.62" x2="342.9" y2="7.62" width="0.1524" layer="91"/>
+<label x="340.36" y="7.62" size="1.778" layer="95"/>
+</segment>
+</net>
+<net name="RX2_UART" class="0">
+<segment>
+<pinref part="U$1" gate="G$1" pin="PA3"/>
+<wire x1="60.96" y1="81.28" x2="83.82" y2="81.28" width="0.1524" layer="91"/>
+<label x="78.74" y="81.28" size="1.778" layer="95"/>
+</segment>
+<segment>
+<wire x1="304.8" y1="2.54" x2="342.9" y2="2.54" width="0.1524" layer="91"/>
+<label x="340.36" y="2.54" size="1.778" layer="95"/>
+</segment>
+</net>
+<net name="RX6_UART" class="0">
+<segment>
+<wire x1="304.8" y1="-2.54" x2="342.9" y2="-2.54" width="0.1524" layer="91"/>
+<label x="340.36" y="-2.54" size="1.778" layer="95"/>
+</segment>
+</net>
+<net name="TX6_UART" class="0">
+<segment>
+<wire x1="304.8" y1="-7.62" x2="342.9" y2="-7.62" width="0.1524" layer="91"/>
+<label x="340.36" y="-7.62" size="1.778" layer="95"/>
+</segment>
+</net>

Commit message: плата
Connections:
- net BUZZER: now also U$1.PA4
- net IRQ_RADIO: now also U$1.PC15; no longer U$1.PB8
- net MOSI_SR: now also U$1.PB5
- net SCL: now also U$1.PB8; no longer U$1.PB6
Changed lines of the file:
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@@
 <label x="340.36" y="88.9" size="1.778" layer="95"/>
+</segment>
+<segment>
+<wire x1="373.38" y1="88.9" x2="411.48" y2="88.9" width="0.1524" layer="91"/>
+<label x="408.94" y="88.9" size="1.778" layer="95"/>
 </segment>
 </net>
@@
 <label x="231.14" y="27.94" size="1.778" layer="95" rot="R90"/>
 </segment>
+<segment>
+<pinref part="U$1" gate="G$1" pin="PA4"/>
+<wire x1="60.96" y1="76.2" x2="83.82" y2="76.2" width="0.1524" layer="91"/>
+<label x="76.2" y="76.2" size="1.778" layer="95"/>
+</segment>
 </net>
 <net name="5V" class="0">
@@
 <wire x1="304.8" y1="99.06" x2="342.9" y2="99.06" width="0.1524" layer="91"/>
 <label x="340.36" y="99.06" size="1.778" layer="95"/>
+</segment>
+<segment>
+<wire x1="373.38" y1="99.06" x2="411.48" y2="99.06" width="0.1524" layer="91"/>
+<label x="408.94" y="99.06" size="1.778" layer="95"/>
 </segment>
 </net>
@@
 <label x="340.36" y="93.98" size="1.778" layer="95"/>
 </segment>
+<segment>
+<wire x1="373.38" y1="93.98" x2="411.48" y2="93.98" width="0.1524" layer="91"/>
+<label x="408.94" y="93.98" size="1.778" layer="95"/>
+</segment>
 </net>
 <net name="SCL" class="0">
@@
 </segment>
 <segment>
-<pinref part="U$1" gate="G$1" pin="PB6"/>
-<wire x1="20.32" y1="71.12" x2="5.08" y2="71.12" width="0.1524" layer="91"/>
-<label x="5.08" y="71.12" size="1.778" layer="95"/>
-</segment>
-<segment>
 <wire x1="304.8" y1="38.1" x2="342.9" y2="38.1" width="0.1524" layer="91"/>
 <label x="340.36" y="38.1" size="1.778" layer="95"/>
+</segment>
+<segment>
+<wire x1="20.32" y1="60.96" x2="5.08" y2="60.96" width="0.1524" layer="91"/>
+<label x="5.08" y="60.96" size="1.778" layer="95"/>
+<pinref part="U$1" gate="G$1" pin="PB8"/>
 </segment>
 </net>
@@
 <label x="340.36" y="12.7" size="1.778" layer="95"/>
 </segment>
+<segment>
+<wire x1="373.38" y1="53.34" x2="411.48" y2="53.34" width="0.1524" layer="91"/>
+<label x="408.94" y="53.34" size="1.778" layer="95"/>
+</segment>
 </net>
 <net name="LATCH_SR" class="0">
@@
 <label x="340.36" y="17.78" size="1.778" layer="95"/>
 </segment>
+<segment>
+<wire x1="373.38" y1="58.42" x2="411.48" y2="58.42" width="0.1524" layer="91"/>
+<label x="408.94" y="58.42" size="1.778" layer="95"/>
+</segment>
 </net>
 <net name="MOSI_SR" class="0">
@@
 <label x="340.36" y="33.02" size="1.778" layer="95"/>
 </segment>
+<segment>
+<wire x1="373.38" y1="68.58" x2="411.48" y2="68.58" width="0.1524" layer="91"/>
+<label x="408.94" y="68.58" size="1.778" layer="95"/>
+</segment>
+<segment>
+<pinref part="U$1" gate="G$1" pin="PB5"/>
+<wire x1="20.32" y1="76.2" x2="0" y2="76.2" width="0.1524" layer="91"/>
+</segment>
 </net>
 <net name="SCK_SR" class="0">
@@
 <label x="340.36" y="27.94" size="1.778" layer="95"/>
 </segment>
+<segment>
+<wire x1="373.38" y1="63.5" x2="411.48" y2="63.5" width="0.1524" layer="91"/>
+<label x="408.94" y="63.5" size="1.778" layer="95"/>
+</segment>
 </net>
 <net name="MOSI_RADIO" class="0">
@@
 </segment>
 </net>
-<net name="IRQ_RADIO" class="0">
-<segment>
-<pinref part="U$1" gate="G$1" pin="PB8"/>
-<wire x1="20.32" y1="60.96" x2="0" y2="60.96" width="0.1524" layer="91"/>
-<label x="0" y="60.96" size="1.778" layer="95"/>
-</segment>
-</net>
 <net name="MISO_SR" class="0">
 <segment>
@@
 <label x="340.36" y="78.74" size="1.778" layer="95"/>
 </segment>
+<segment>
+<wire x1="373.38" y1="78.74" x2="411.48" y2="78.74" width="0.1524" layer="91"/>
+<label x="408.94" y="78.74" size="1.778" layer="95"/>
+</segment>
 </net>
 <net name="TX_UART" class="0">
@@
 <label x="340.36" y="73.66" size="1.778" layer="95"/>
 </segment>
+<segment>
+<wire x1="373.38" y1="73.66" x2="411.48" y2="73.66" width="0.1524" layer="91"/>
+<label x="408.94" y="73.66" size="1.778" layer="95"/>
+</segment>
 </net>
 <net name="MISO_RADIO" class="0">
@@
 <label x="340.36" y="83.82" size="1.778" layer="95"/>
 </segment>
+<segment>
+<wire x1="373.38" y1="83.82" x2="411.48" y2="83.82" width="0.1524" layer="91"/>
+<label x="408.94" y="83.82" size="1.778" layer="95"/>
+</segment>
 </net>
 <net name="CE_RADIO" class="0">
@@
 <label x="340.36" y="7.62" size="1.778" layer="95"/>
 </segment>
+<segment>
+<wire x1="373.38" y1="48.26" x2="411.48" y2="48.26" width="0.1524" layer="91"/>
+<label x="408.94" y="48.26" size="1.778" layer="95"/>
+</segment>
 </net>
 <net name="RX2_UART" class="0">
@@
 <label x="340.36" y="2.54" size="1.778" layer="95"/>
 </segment>
+<segment>
+<wire x1="373.38" y1="43.18" x2="411.48" y2="43.18" width="0.1524" layer="91"/>
+<label x="408.94" y="43.18" size="1.778" layer="95"/>
+</segment>
 </net>
 <net name="RX6_UART" class="0">
@@
 </segment>
 </net>
+<net name="N$3" class="0">
+<segment>
+<wire x1="198.12" y1="68.58" x2="198.12" y2="71.12" width="0.1524" layer="91"/>
+</segment>
+</net>
+<net name="IRQ_RADIO" class="0">
+<segment>
+<pinref part="U$1" gate="G$1" pin="PC15"/>
+<wire x1="20.32" y1="15.24" x2="0" y2="15.24" width="0.1524" layer="91"/>
+<label x="0" y="15.24" size="1.778" layer="95"/>
+</segment>
+</net>

Commit message: разъемы смд
Parts:
- added U$3: PBS_SMD_X12, UNKNOWN-2024:PBS_SMD_X12
- added U$4: PBS_SMD_X9, UNKNOWN-2024:PBS_SMD_X9
Connections:
- net RX2_UART renamed RX2_BLE
- net RX_UART renamed RX1_GPS
- net TX2_UART renamed TX2_BLE
- net TX_UART renamed TX1_GPS
- new net DIR_DRIVER: U$1.PA9
- new net STEP_DRIVER: U$1.PA10
- new net SW_AMP: U$1.PB6

Commit message: разъемы еще
Parts:
- removed U$4: PBS_SMD_X9, UNKNOWN-2024:PBS_SMD_X9
- added U$5: STM32F411_BOARD, UNKNOWN-2024:STM32F411_BOARD
- U$1: value BLACKPILL -> PBS_SMD_X13; device UNKNOWN-2024:BLACKPILL -> UNKNOWN-2024:PBS_SMD_X13
- U$3: value PBS_SMD_X12 -> PBS_SMD_X9; device UNKNOWN-2024:PBS_SMD_X12 -> UNKNOWN-2024:PBS_SMD_X9
Connections:
- removed net CMD: MICRO_SD.CMD, U$1.PA6
- removed net RX1_GPS: U$1.PB3
- removed net RX2_BLE: U$1.PA3
- removed net SD_CLK: MICRO_SD.CLK, U$1.PB15
- removed net TX1_GPS: U$1.PA15
- removed net TX2_BLE: U$1.PA2
- new net CMD_SD: MICRO_SD.CMD, U$5.PA6
- new net RX1_BLE: U$1.4, U$5.PB3
- new net RX2_GPS: U$3.8, U$5.PA3
- new net SD_CK: MICRO_SD.CLK, U$5.PB15
- new net TX1_BLE: U$1.3, U$5.PA15
- new net TX2_GPS: U$3.7, U$5.PA2
- net 3V3: now also U$1.13, U$5.3V3, U$5.VBAT; no longer U$1.3V3
- net 5V: now also U$1.11, U$5.5V; no longer U$1.5V
- net ADC_FOTO: now also U$1.10, U$5.PA0; no longer U$1.PA0
- net BUZZER: now also U$5.PB0; no longer U$1.PA4
- net CE_RADIO: now also U$3.1, U$5.PC13; no longer U$1.PC13
- net CS_RADIO: now also U$3.2, U$5.PC14; no longer U$1.PC14
- net D0_SD: now also U$5.PB7; no longer U$1.PB7
- net DIR_DRIVER: now also U$1.1, U$5.PA9; no longer U$1.PA9
- net GND: now also U$1.12, U$5.GND; no longer U$1.GND
- net IRQ_RADIO: now also U$3.3, U$5.PC15; no longer U$1.PC15
- net LATCH_SR: now also U$1.5, U$5.PB12; no longer U$1.PB2
- net MISO_RADIO: now also U$3.5, U$5.PA11; no longer U$1.PA11
- net MISO_SR: now also U$1.8, U$5.PB4; no longer U$1.PB4
- net MOSI_RADIO: now also U$3.4, U$5.PA1; no longer U$1.PA1
- net MOSI_SR: now also U$1.9, U$5.PB5; no longer U$1.PA7, U$1.PB5
- net OE_SR: now also U$1.6, U$5.PB14; no longer U$1.PB10
- net SCK_RADIO: now also U$3.6, U$5.PB13; no longer U$1.PB13
- net SCK_SR: now also U$1.7, U$5.PA5; no longer U$1.PA5
- net SCL: now also U$5.PB8; no longer U$1.PB8
- net SDA: now also U$5.PB9; no longer U$1.PB9
- net STEP_DRIVER: now also U$1.2, U$5.PA10; no longer U$1.PA10
- net SWITCH: now also U$5.PB1; no longer U$1.PB1
- net SW_AMP: now also U$3.9, U$5.PA4; no longer U$1.PB6

Commit message: плата МК под разводку
Parts:
- removed U$1: PBS_SMD_X13, UNKNOWN-2024:PBS_SMD_X13
- removed U$3: PBS_SMD_X9, UNKNOWN-2024:PBS_SMD_X9
- added U$4: PBS_SMD_X13, UNKNOWN-2024:PBS_SMD_X13
- added U$6: PBS_SMD_X9, UNKNOWN-2024:PBS_SMD_X9
- BME280: value BME280 -> BME280BME280-PINS-ONLY; device UNKNOWN-2024:BME280 -> UNKNOWN-2024:BME280BME280-PINS-ONLY
Connections:
- removed net D0: MICRO_SD.DAT0
- net 3V3: now also U$4.1; no longer U$1.13
- net 5V: now also U$4.3; no longer U$1.11
- net ADC_FOTO: now also U$4.4; no longer U$1.10
- net CE_RADIO: now also U$6.9; no longer U$3.1
- net CS_RADIO: now also U$6.8; no longer U$3.2
- net D0_SD: now also MICRO_SD.DAT0
- net DIR_DRIVER: now also U$4.13; no longer U$1.1
- net GND: now also U$4.2; no longer U$1.12
- net IRQ_RADIO: now also U$6.7; no longer U$3.3
- net LATCH_SR: now also U$4.9, U$5.PB14; no longer U$1.5, U$5.PB12
- net MISO_RADIO: now also U$6.5; no longer U$3.5
- net MISO_SR: now also U$4.6; no longer U$1.8
- net MOSI_RADIO: now also U$6.6; no longer U$3.4
- net MOSI_SR: now also U$4.5; no longer U$1.9
- net OE_SR: now also U$4.8, U$5.PA8; no longer U$1.6, U$5.PB14
- net RX1_BLE: now also U$4.10; no longer U$1.4
- net RX2_GPS: now also U$6.2; no longer U$3.8
- net SCK_RADIO: now also U$6.4; no longer U$3.6
- net SCK_SR: now also U$4.7; no longer U$1.7
- net STEP_DRIVER: now also U$4.12; no longer U$1.2
- net SWITCH: now also U$5.PB12; no longer U$5.PB1
- net SW_AMP: now also U$6.1; no longer U$3.9
- net TX1_BLE: now also U$4.11; no longer U$1.3
- net TX2_GPS: now also U$6.3; no longer U$3.7
Other:
- moved on the sheet: BME280

Commit message: sdfghgfds
Parts:
- added C1: (no value), rcl:C-EUC0603
- added R3, R4: 5k1, rcl:R-US_R0603
- added R5, R6: 10k, rcl:R-US_R0603
Connections:
- net 3V3: now also C1.2, R3.2, R4.2, R5.1, R6.1
- net CMD_SD: now also R6.2
- net D0_SD: now also R5.2
- net GND: now also C1.1
- net SCL: now also R4.1
- net SDA: now also R3.1
Changed lines of the file:
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@@
 <?xml version="1.0" encoding="utf-8"?>
 <!DOCTYPE eagle SYSTEM "eagle.dtd">
-<eagle version="9.6.2">
+<eagle version="9.6.0">
 <drawing>
 <settings>
@@
 <part name="U$4" library="UNKNOWN-2024" deviceset="PBS_SMD_X13" device=""/>
 <part name="U$6" library="UNKNOWN-2024" deviceset="PBS_SMD_X9" device=""/>
+<part name="R3" library="rcl" library_urn="urn:adsk.eagle:library:334" deviceset="R-US_" device="R0603" package3d_urn="urn:adsk.eagle:package:23555/3" value="5k1"/>
+<part name="R4" library="rcl" library_urn="urn:adsk.eagle:library:334" deviceset="R-US_" device="R0603" package3d_urn="urn:adsk.eagle:package:23555/3" value="5k1"/>
+<part name="R5" library="rcl" library_urn="urn:adsk.eagle:library:334" deviceset="R-US_" device="R0603" package3d_urn="urn:adsk.eagle:package:23555/3" value="10k"/>
+<part name="R6" library="rcl" library_urn="urn:adsk.eagle:library:334" deviceset="R-US_" device="R0603" package3d_urn="urn:adsk.eagle:package:23555/3" value="10k"/>
+<part name="C1" library="rcl" library_urn="urn:adsk.eagle:library:334" deviceset="C-EU" device="C0603" package3d_urn="urn:adsk.eagle:package:23616/2"/>
 </parts>
 <sheets>
@@
 <attribute name="VALUE" x="72.39" y="25.4" size="1.778" layer="96"/>
 </instance>
+<instance part="R3" gate="G$1" x="-93.98" y="45.72" smashed="yes" rot="R180">
+<attribute name="NAME" x="-90.17" y="44.2214" size="1.778" layer="95" rot="R180"/>
+<attribute name="VALUE" x="-97.79" y="43.942" size="1.778" layer="96" rot="R180"/>
+</instance>
+<instance part="R4" gate="G$1" x="-93.98" y="48.26" smashed="yes" rot="R180">
+<attribute name="NAME" x="-90.17" y="51.8414" size="1.778" layer="95" rot="R180"/>
+<attribute name="VALUE" x="-97.79" y="51.562" size="1.778" layer="96" rot="R180"/>
+</instance>
+<instance part="R5" gate="G$1" x="167.64" y="104.14" smashed="yes" rot="R180">
+<attribute name="NAME" x="171.45" y="102.6414" size="1.778" layer="95" rot="R180"/>
+<attribute name="VALUE" x="171.45" y="107.442" size="1.778" layer="96" rot="R180"/>
+</instance>
+<instance part="R6" gate="G$1" x="167.64" y="91.44" smashed="yes" rot="R180">
+<attribute name="NAME" x="171.45" y="89.9414" size="1.778" layer="95" rot="R180"/>
+<attribute name="VALUE" x="171.45" y="94.742" size="1.778" layer="96" rot="R180"/>
+</instance>
+<instance part="C1" gate="G$1" x="165.1" y="99.06" smashed="yes">
+<attribute name="NAME" x="166.624" y="99.441" size="1.778" layer="95"/>
+<attribute name="VALUE" x="166.624" y="94.361" size="1.778" layer="96"/>
+</instance>
 </instances>
 <busses>
@@
 <segment>
 <pinref part="MICRO_SD" gate="G$1" pin="VSS"/>
-<wire x1="149.86" y1="99.06" x2="165.1" y2="99.06" width="0.1524" layer="91"/>
-<label x="157.48" y="99.06" size="1.778" layer="95"/>
+<wire x1="149.86" y1="99.06" x2="162.56" y2="99.06" width="0.1524" layer="91"/>
+<label x="152.4" y="99.06" size="1.778" layer="95"/>
+<pinref part="C1" gate="G$1" pin="1"/>
+<wire x1="165.1" y1="101.6" x2="162.56" y2="101.6" width="0.1524" layer="91"/>
+<wire x1="162.56" y1="101.6" x2="162.56" y2="99.06" width="0.1524" layer="91"/>
 </segment>
 <segment>
@@
 <pinref part="MICRO_SD" gate="G$1" pin="VDD"/>
 <wire x1="149.86" y1="93.98" x2="165.1" y2="93.98" width="0.1524" layer="91"/>
-<label x="157.48" y="93.98" size="1.778" layer="95"/>
+<label x="152.4" y="93.98" size="1.778" layer="95"/>
+<pinref part="C1" gate="G$1" pin="2"/>
 </segment>
 <segment>
@@
 <segment>
 <pinref part="U$5" gate="G$1" pin="3V3"/>
-<wire x1="-68.58" y1="38.1" x2="-88.9" y2="38.1" width="0.1524" layer="91"/>
+<wire x1="-68.58" y1="38.1" x2="-99.06" y2="38.1" width="0.1524" layer="91"/>
 <label x="-88.9" y="38.1" size="1.778" layer="95"/>
+<pinref part="R3" gate="G$1" pin="2"/>
+<wire x1="-99.06" y1="38.1" x2="-99.06" y2="45.72" width="0.1524" layer="91"/>
+<pinref part="R4" gate="G$1" pin="2"/>
+<wire x1="-99.06" y1="48.26" x2="-99.06" y2="45.72" width="0.1524" layer="91"/>
+<junction x="-99.06" y="45.72"/>
 </segment>
 <segment>
@@
 </segment>
 <segment>
-<wire x1="200.66" y1="104.14" x2="187.96" y2="104.14" width="0.1524" layer="91"/>
 <label x="187.96" y="104.14" size="1.778" layer="95"/>
 <pinref part="BME280" gate="G$1" pin="VIN"/>
+<pinref part="R5" gate="G$1" pin="1"/>
+<pinref part="R6" gate="G$1" pin="1"/>
+<wire x1="172.72" y1="104.14" x2="172.72" y2="91.44" width="0.1524" layer="91"/>
+<wire x1="172.72" y1="104.14" x2="200.66" y2="104.14" width="0.1524" layer="91"/>
+<junction x="172.72" y="104.14"/>
 </segment>
 <segment>
@@
 <label x="-88.9" y="48.26" size="1.778" layer="95"/>
 <pinref part="U$5" gate="G$1" pin="PB8"/>
+<pinref part="R4" gate="G$1" pin="1"/>
 </segment>
 <segment>
@@
 <label x="-88.9" y="45.72" size="1.778" layer="95"/>
 <pinref part="U$5" gate="G$1" pin="PB9"/>
+<pinref part="R3" gate="G$1" pin="1"/>
 </segment>
 <segment>
@@
 <segment>
 <pinref part="MICRO_SD" gate="G$1" pin="CMD"/>
-<wire x1="149.86" y1="91.44" x2="165.1" y2="91.44" width="0.1524" layer="91"/>
-<label x="157.48" y="91.44" size="1.778" layer="95"/>
+<wire x1="149.86" y1="91.44" x2="162.56" y2="91.44" width="0.1524" layer="91"/>
+<label x="152.4" y="91.44" size="1.778" layer="95"/>
+<pinref part="R6" gate="G$1" pin="2"/>
 </segment>
 <segment>
@@
 <segment>
 <pinref part="MICRO_SD" gate="G$1" pin="CLK"/>
-<wire x1="149.86" y1="96.52" x2="165.1" y2="96.52" width="0.1524" layer="91"/>
-<label x="157.48" y="96.52" size="1.778" layer="95"/>
+<wire x1="149.86" y1="96.52" x2="162.56" y2="96.52" width="0.1524" layer="91"/>
+<label x="152.4" y="96.52" size="1.778" layer="95"/>
 </segment>
 <segment>
@@
 <segment>
 <pinref part="MICRO_SD" gate="G$1" pin="DAT0"/>
-<wire x1="149.86" y1="101.6" x2="165.1" y2="101.6" width="0.1524" layer="91"/>
-<label x="157.48" y="101.6" size="1.778" layer="95"/>
+<label x="152.4" y="101.6" size="1.778" layer="95"/>
+<pinref part="R5" gate="G$1" pin="2"/>
+<wire x1="162.56" y1="104.14" x2="157.48" y2="104.14" width="0.1524" layer="91"/>
+<wire x1="157.48" y1="104.14" x2="157.48" y2="101.6" width="0.1524" layer="91"/>
+<wire x1="157.48" y1="101.6" x2="149.86" y2="101.6" width="0.1524" layer="91"/>
 </segment>
 </net>
@@
 packages will not be understood (or retained) with this version.
 </note>
+<note version="8.4" severity="warning">
+Since Version 8.4, EAGLE supports properties for SPICE simulation.
+Probes in schematics and SPICE mapping objects found in parts and library devices
+will not be understood with this version. Update EAGLE to the latest version
+for full support of SPICE simulation.
+</note>
 </compatibility>
