File: schematics/KPNN2024/Board/pitanie.sch (EAGLE design)
At the start: 36 parts

Commit message: отртамгор
Parts:
- removed LIS: LIS3MDL-GY, CanCubeSat:LIS3MDL-GY
Connections:
- new net CE_RADIO: U$9.1
- new net CS_RADIO: U$9.2
- new net IRQ_RADIO: U$9.3
- new net MISO_RADIO: U$9.5
- new net MOSI_RADIO: U$9.4
- new net RX1_BLF: U$10.4
- new net RX2_GPS: U$9.8
- new net SCK_RADIO: U$9.6
- new net SW_AMP: U$9.9
- new net TX1_BLF: U$10.3
- new net TX2_GPS: U$9.7
- net 3V3: now also U$10.13
- net 5V: now also U$10.11
- net DIR_DRIVER: now also U$10.1
- net FOTO: now also U$10.10
- net GND: now also U$10.12
- net LATCH_SR: now also U$10.5
- net MISO_SR: now also U$10.8
- net MOSI_SR: now also U$10.9
- net OE_SR: now also U$10.6
- net SCK_SR: now also U$10.7
- net STEP_DRIVER: now also U$10.2
Changed lines of the file:
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@@
 <part name="U$8" library="KNPN-2023" deviceset="VT93N1" device=""/>
 <part name="LSM" library="UNKNOWN-2024" deviceset="LSM6DS3-GY" device=""/>
-<part name="LIS" library="CanCubeSat" deviceset="LIS3MDL-GY" device=""/>
 <part name="R7" library="rcl" library_urn="urn:adsk.eagle:library:334" deviceset="R-US_" device="R0603" package3d_urn="urn:adsk.eagle:package:23555/3" value="2k"/>
 <part name="TMC" library="UNKNOWN-2024" deviceset="DRIVER_TMC2209" device=""/>
@@
 <instance part="LSM" gate="G$1" x="193.04" y="167.64" smashed="yes">
 <attribute name="NAME" x="185.42" y="185.42" size="1.778" layer="95"/>
-</instance>
-<instance part="LIS" gate="G$1" x="193.04" y="116.84" smashed="yes">
-<attribute name="NAME" x="185.42" y="134.62" size="1.778" layer="95"/>
 </instance>
 <instance part="R7" gate="G$1" x="119.38" y="88.9" smashed="yes" rot="R90">
@@
 <label x="83.82" y="160.02" size="1.778" layer="95"/>
 </segment>
+<segment>
+<pinref part="U$10" gate="G$1" pin="13"/>
+<wire x1="388.62" y1="7.62" x2="365.76" y2="7.62" width="0.1524" layer="91"/>
+<label x="365.76" y="7.62" size="1.778" layer="95"/>
+</segment>
 </net>
 <net name="BUS+" class="0">
@@
 <label x="40.64" y="142.24" size="1.778" layer="95"/>
 </segment>
+<segment>
+<pinref part="U$10" gate="G$1" pin="12"/>
+<wire x1="388.62" y1="10.16" x2="365.76" y2="10.16" width="0.1524" layer="91"/>
+<label x="365.76" y="10.16" size="1.778" layer="95"/>
+</segment>
 </net>
 <net name="8V" class="0">
@@
 <label x="134.62" y="96.52" size="1.778" layer="95"/>
 </segment>
+<segment>
+<pinref part="U$10" gate="G$1" pin="10"/>
+<wire x1="388.62" y1="15.24" x2="365.76" y2="15.24" width="0.1524" layer="91"/>
+<label x="365.76" y="15.24" size="1.778" layer="95"/>
+</segment>
 </net>
 <net name="OE_SR" class="0">
@@
 <wire x1="78.74" y1="152.4" x2="88.9" y2="152.4" width="0.1524" layer="91"/>
 <label x="83.82" y="152.4" size="1.778" layer="95"/>
+</segment>
+<segment>
+<pinref part="U$10" gate="G$1" pin="6"/>
+<wire x1="388.62" y1="25.4" x2="365.76" y2="25.4" width="0.1524" layer="91"/>
+<label x="365.76" y="25.4" size="1.778" layer="95"/>
 </segment>
 </net>
@@
 <label x="395.55" y="96.6" size="1.778" layer="95"/>
 </segment>
+<segment>
+<pinref part="U$10" gate="G$1" pin="11"/>
+<wire x1="388.62" y1="12.7" x2="365.76" y2="12.7" width="0.1524" layer="91"/>
+<label x="365.76" y="12.7" size="1.778" layer="95"/>
+</segment>
 </net>
 <net name="LATCH_SR" class="0">
@@
 <label x="78.74" y="149.86" size="1.778" layer="95"/>
 </segment>
+<segment>
+<pinref part="U$10" gate="G$1" pin="5"/>
+<wire x1="388.62" y1="27.94" x2="365.76" y2="27.94" width="0.1524" layer="91"/>
+<label x="365.76" y="27.94" size="1.778" layer="95"/>
+</segment>
 </net>
 <net name="SCK_SR" class="0">
@@
 <label x="86.36" y="147.32" size="1.778" layer="95"/>
 </segment>
+<segment>
+<pinref part="U$10" gate="G$1" pin="7"/>
+<wire x1="388.62" y1="22.86" x2="365.76" y2="22.86" width="0.1524" layer="91"/>
+<label x="365.76" y="22.86" size="1.778" layer="95"/>
+</segment>
 </net>
 <net name="MOSI_SR" class="0">
@@
 <wire x1="78.74" y1="154.94" x2="88.9" y2="154.94" width="0.1524" layer="91"/>
 <label x="86.36" y="154.94" size="1.778" layer="95"/>
+</segment>
+<segment>
+<pinref part="U$10" gate="G$1" pin="9"/>
+<wire x1="388.62" y1="17.78" x2="365.76" y2="17.78" width="0.1524" layer="91"/>
+<label x="365.76" y="17.78" size="1.778" layer="95"/>
 </segment>
 </net>
@@
 <label x="336.296" y="82.55" size="1.778" layer="95"/>
 </segment>
+<segment>
+<pinref part="U$10" gate="G$1" pin="2"/>
+<wire x1="388.62" y1="35.56" x2="365.76" y2="35.56" width="0.1524" layer="91"/>
+<label x="365.76" y="35.56" size="1.778" layer="95"/>
+</segment>
 </net>
 <net name="DIR_DRIVER" class="0">
@@
 <label x="336.55" y="79.756" size="1.778" layer="95"/>
 </segment>
+<segment>
+<pinref part="U$10" gate="G$1" pin="1"/>
+<wire x1="388.62" y1="38.1" x2="365.76" y2="38.1" width="0.1524" layer="91"/>
+<label x="365.76" y="38.1" size="1.778" layer="95"/>
+</segment>
 </net>
 <net name="MISO_SR" class="0">
@@
 <label x="220.98" y="152.4" size="1.778" layer="95"/>
 </segment>
-</net>
+<segment>
+<pinref part="U$10" gate="G$1" pin="8"/>
+<wire x1="388.62" y1="20.32" x2="365.76" y2="20.32" width="0.1524" layer="91"/>
+<label x="365.76" y="20.32" size="1.778" layer="95"/>
+</segment>
+</net>
+<net name="CE_RADIO" class="0">
+<segment>
+<pinref part="U$9" gate="G$1" pin="1"/>
+<wire x1="337.82" y1="38.1" x2="317.5" y2="38.1" width="0.1524" layer="91"/>
+<label x="317.5" y="38.1" size="1.778" layer="95"/>
+</segment>
+</net>
+<net name="CS_RADIO" class="0">
+<segment>
+<pinref part="U$9" gate="G$1" pin="2"/>
+<wire x1="337.82" y1="35.56" x2="317.5" y2="35.56" width="0.1524" layer="91"/>
+<label x="317.5" y="35.56" size="1.778" layer="95"/>
+</segment>
+</net>
+<net name="IRQ_RADIO" class="0">
+<segment>
+<pinref part="U$9" gate="G$1" pin="3"/>
+<wire x1="337.82" y1="33.02" x2="317.5" y2="33.02" width="0.1524" layer="91"/>
+<label x="317.5" y="33.02" size="1.778" layer="95"/>
+</segment>
+</net>
+<net name="MOSI_RADIO" class="0">
+<segment>
+<pinref part="U$9" gate="G$1" pin="4"/>
+<wire x1="337.82" y1="30.48" x2="317.5" y2="30.48" width="0.1524" layer="91"/>
+<label x="317.5" y="30.48" size="1.778" layer="95"/>
+</segment>
+</net>
+<net name="MISO_RADIO" class="0">
+<segment>
+<pinref part="U$9" gate="G$1" pin="5"/>
+<wire x1="337.82" y1="27.94" x2="317.5" y2="27.94" width="0.1524" layer="91"/>
+<label x="317.5" y="27.94" size="1.778" layer="95"/>
+</segment>
+</net>
+<net name="SCK_RADIO" class="0">
+<segment>
+<pinref part="U$9" gate="G$1" pin="6"/>
+<wire x1="337.82" y1="25.4" x2="317.5" y2="25.4" width="0.1524" layer="91"/>
+<label x="317.5" y="25.4" size="1.778" layer="95"/>
+</segment>
+</net>
+<net name="TX2_GPS" class="0">
+<segment>
+<pinref part="U$9" gate="G$1" pin="7"/>
+<wire x1="337.82" y1="22.86" x2="317.5" y2="22.86" width="0.1524" layer="91"/>
+<label x="317.5" y="22.86" size="1.778" layer="95"/>
+</segment>
+</net>
+<net name="RX2_GPS" class="0">
+<segment>
+<pinref part="U$9" gate="G$1" pin="8"/>
+<wire x1="337.82" y1="20.32" x2="317.5" y2="20.32" width="0.1524" layer="91"/>
+<label x="317.5" y="20.32" size="1.778" layer="95"/>
+</segment>
+</net>
+<net name="SW_AMP" class="0">
+<segment>
+<pinref part="U$9" gate="G$1" pin="9"/>
+<wire x1="337.82" y1="17.78" x2="317.5" y2="17.78" width="0.1524" layer="91"/>
+<label x="317.5" y="17.78" size="1.778" layer="95"/>
+</segment>
+</net>
+<net name="TX1_BLF" class="0">
+<segment>
+<pinref part="U$10" gate="G$1" pin="3"/>
+<wire x1="388.62" y1="33.02" x2="365.76" y2="33.02" width="0.1524" layer="91"/>
+<label x="365.76" y="33.02" size="1.778" layer="95"/>
+</segment>
+</net>
+<net name="RX1_BLF" class="0">
+<segment>
+<pinref part="U$10" gate="G$1" pin="4"/>
+<wire x1="388.62" y1="30.48" x2="365.76" y2="30.48" width="0.1524" layer="91"/>
+<label x="365.76" y="30.48" size="1.778" layer="95"/>
+</segment>
+</net>

Commit message: Добавлены разъемы на плату питания
Parts:
- removed TMC: DRIVER_TMC2209, UNKNOWN-2024:DRIVER_TMC2209
- added R10, R8: 10k, rcl:R-US_R0603
- added R9: 100R, rcl:R-US_R0603
- added U$12: IRF7905PBF, UNKNOWN-2024:IRF7905PBF
- added U$13: TMC2209_WITHOUT, UNKNOWN-2024:TMC2209_WITHOUT
- added U$14: MOLEX-4-1.25, UNKNOWN-2024:MOLEX-4-1.25
- added X1, X2: JST-2-2.5, UNKNOWN-2024:JST-2-2.5
- LSM: value LSM6DS3-GY -> LSM6DS3_WITHOUT; device UNKNOWN-2024:LSM6DS3-GY -> UNKNOWN-2024:LSM6DS3_WITHOUT
- U$9: value PBS_SMD_X9 -> JST-4-2.5; device UNKNOWN-2024:PBS_SMD_X9 -> UNKNOWN-2024:JST-4-2.5
Connections:
- removed net 8V: S1.S
- removed net CE_RADIO: U$9.1
- removed net CS_RADIO: U$9.2
- removed net GND-OUT: C1.1, C10.1, C13.1, C14.1, C2.1, C3.1, C6.1, C7.1, C8.1, C9.1, R2.2, R5.2, U$1.IN-, U$1.OUT-, U$2.AGND, U$2.GND, U$4.IN-, U$4.OUT-, U$5.AGND, U$5.GND
- removed net IRQ_RADIO: U$9.3
- removed net MISO_RADIO: U$9.5
- removed net MOSI_RADIO: U$9.4
- removed net RX1_BLF: U$10.4
- removed net RX2_GPS: U$9.8
- removed net SCK_RADIO: U$9.6
- removed net SW_AMP: U$9.9
- removed net TX1_BLF: U$10.3
- removed net TX2_GPS: U$9.7
- new net A1: U$13.A1, U$9.1
- new net A2: U$13.A2, U$9.3
- new net B1: U$13.B1, U$9.2
- new net B2: U$13.B2, U$9.4
- new net BUS+_OUT: S1.O, X2.2
- new net EN_DRIVER: U$13.EN
- new net N$6: R10.2, R9.1, U$12.G2
- new net PERE_G: U$12.S2, X1.2
- new net Q2: R9.2
- new net RX1_BLE: U$10.4, U$14.3
- new net TX1_BLE: U$10.3, U$14.4
- new net VCC: U$14.1
- net 3V3: now also R8.2, U$13.VDD, U$7.MR; no longer C12.1, C13.2, C14.2, R6.2, U$4.OUT+, U$6.1
- net 5V: now also C12.1, C13.2, C14.2, R6.2, U$13.VM, U$4.OUT+, U$6.1; no longer TMC.P$16
- net BUS+: now also S1.P, X1.1
- net DIR_DRIVER: now also U$13.DIR; no longer TMC.P$8
- net GND: now also C1.1, C10.1, C13.1, C14.1, C2.1, C3.1, C6.1, C7.1, C8.1, C9.1, R10.1, R2.2, R5.2, U$1.IN-, U$1.OUT-, U$12.D2, U$13.GND, U$13.GND_, U$14.2, U$2.AGND, U$2.GND, U$4.IN-, U$4.OUT-, U$5.AGND, U$5.GND, X2.1; no longer S1.O, TMC.P$15, TMC.P$9
- net OE_SR: now also R8.1
- net STEP_DRIVER: now also U$13.STEP; no longer TMC.P$7
Other:
- moved on the sheet: R4

Commit message: Разведена плата питания
Connections:
- removed net BUZZER: U$7.Q7
- removed net Q1: U$11.CS, U$7.Q1
- removed net Q2: R9.2
- removed net Q4: LSM.CS, U$7.Q4
- removed net VCC: U$14.1
- new net CS_LIS: U$11.CS, U$7.Q2
- new net CS_LSM: LSM.CS, U$7.Q6
- new net PERE: R9.2, U$7.Q1
- net 5V: now also U$14.1
- net EN_DRIVER: now also U$7.Q7
Changed lines of the file:
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@@
 <segment>
 <pinref part="U$7" gate="G$1" pin="GND"/>
-<wire x1="53.34" y1="142.24" x2="40.64" y2="142.24" width="0.1524" layer="91"/>
-<label x="40.64" y="142.24" size="1.778" layer="95"/>
+<wire x1="53.34" y1="142.24" x2="38.1" y2="142.24" width="0.1524" layer="91"/>
+<label x="38.1" y="142.24" size="1.778" layer="95"/>
 </segment>
 <segment>
@@
 </segment>
 </net>
-<net name="Q1" class="0">
+<net name="PERE" class="0">
 <segment>
 <pinref part="U$7" gate="G$1" pin="Q1"/>
-<wire x1="53.34" y1="160.02" x2="40.64" y2="160.02" width="0.1524" layer="91"/>
-<label x="40.64" y="160.02" size="1.778" layer="95"/>
-</segment>
-<segment>
-<label x="228.6" y="101.6" size="1.778" layer="95"/>
-<pinref part="U$11" gate="G$1" pin="CS"/>
-<wire x1="241.3" y1="101.6" x2="228.6" y2="101.6" width="0.1524" layer="91"/>
-</segment>
-</net>
-<net name="Q4" class="0">
-<segment>
-<pinref part="U$7" gate="G$1" pin="Q4"/>
-<wire x1="53.34" y1="152.4" x2="40.64" y2="152.4" width="0.1524" layer="91"/>
-<label x="40.64" y="152.4" size="1.778" layer="95"/>
-</segment>
-<segment>
-<pinref part="LSM" gate="G$1" pin="CS"/>
-<wire x1="208.28" y1="157.48" x2="223.52" y2="157.48" width="0.1524" layer="91"/>
-<label x="215.9" y="157.48" size="1.778" layer="95"/>
-</segment>
-</net>
-<net name="BUZZER" class="0">
-<segment>
-<pinref part="U$7" gate="G$1" pin="Q7"/>
-<wire x1="53.34" y1="144.78" x2="40.64" y2="144.78" width="0.1524" layer="91"/>
-<label x="40.64" y="144.78" size="1.778" layer="95"/>
+<wire x1="53.34" y1="160.02" x2="38.1" y2="160.02" width="0.1524" layer="91"/>
+<label x="38.1" y="160.02" size="1.778" layer="95"/>
+</segment>
+<segment>
+<pinref part="R9" gate="G$1" pin="2"/>
+<wire x1="38.1" y1="124.46" x2="38.1" y2="132.08" width="0.1524" layer="91"/>
+<label x="38.1" y="127" size="1.778" layer="95" rot="R90"/>
 </segment>
 </net>
@@
 <label x="408.94" y="96.52" size="1.778" layer="95"/>
 </segment>
+<segment>
+<pinref part="U$14" gate="G$1" pin="1"/>
+<wire x1="447.04" y1="45.72" x2="462.28" y2="45.72" width="0.1524" layer="91"/>
+<label x="454.66" y="45.72" size="1.778" layer="95"/>
+</segment>
 </net>
 <net name="LATCH_SR" class="0">
@@
 </segment>
 </net>
-<net name="Q2" class="0">
-<segment>
-<pinref part="R9" gate="G$1" pin="2"/>
-<wire x1="38.1" y1="124.46" x2="38.1" y2="132.08" width="0.1524" layer="91"/>
-<label x="38.1" y="129.54" size="1.778" layer="95" rot="R90"/>
+<net name="CS_LIS" class="0">
+<segment>
+<pinref part="U$7" gate="G$1" pin="Q2"/>
+<wire x1="53.34" y1="157.48" x2="38.1" y2="157.48" width="0.1524" layer="91"/>
+<label x="38.1" y="157.48" size="1.778" layer="95"/>
+</segment>
+<segment>
+<label x="228.6" y="101.6" size="1.778" layer="95"/>
+<pinref part="U$11" gate="G$1" pin="CS"/>
+<wire x1="241.3" y1="101.6" x2="228.6" y2="101.6" width="0.1524" layer="91"/>
 </segment>
 </net>
@@
 <label x="342.9" y="96.52" size="1.778" layer="95"/>
 </segment>
+<segment>
+<pinref part="U$7" gate="G$1" pin="Q7"/>
+<wire x1="53.34" y1="144.78" x2="38.1" y2="144.78" width="0.1524" layer="91"/>
+<label x="38.1" y="144.78" size="1.778" layer="95"/>
+</segment>
 </net>
 <net name="TX1_BLE" class="0">
@@
 <wire x1="388.62" y1="30.48" x2="365.76" y2="30.48" width="0.1524" layer="91"/>
 <label x="365.76" y="30.48" size="1.778" layer="95"/>
-</segment>
-</net>
-<net name="VCC" class="0">
-<segment>
-<pinref part="U$14" gate="G$1" pin="1"/>
-<wire x1="447.04" y1="45.72" x2="462.28" y2="45.72" width="0.1524" layer="91"/>
-<label x="454.66" y="45.72" size="1.778" layer="95"/>
 </segment>
 </net>
@@
 </segment>
 </net>
+<net name="CS_LSM" class="0">
+<segment>
+<pinref part="U$7" gate="G$1" pin="Q6"/>
+<wire x1="53.34" y1="147.32" x2="38.1" y2="147.32" width="0.1524" layer="91"/>
+<label x="38.1" y="147.32" size="1.778" layer="95"/>
+</segment>
+<segment>
+<pinref part="LSM" gate="G$1" pin="CS"/>
+<wire x1="208.28" y1="157.48" x2="223.52" y2="157.48" width="0.1524" layer="91"/>
+<label x="215.9" y="157.48" size="1.778" layer="95"/>
+</segment>
+</net>
