File: schematics/KPNN2024/Board/RADIO.brd (EAGLE design)
At the start: 68.2 x 68.2 mm, 7 parts, among them J1 U.FL-R-SMT-1_10_, J2 U.FL-R-SMT-1_10_

Commit message: SUS
Parts:
- added U$6: PBS_SMD_X13, UNKNOWN-2024:PBD_SMD_X13
- added U$7: PBS_SMD_X9, UNKNOWN-2024:PBS_SMD_X9
- moved U$1 46.9 mm to (50.9, 64.0), turned to 270 degrees
- moved U$2 35.2 mm to (58.7, 63.9), turned to 180 degrees
- moved U$4 23.6 mm to (25.7, 33.1), turned to 0 degrees
- moved U$5 20.1 mm to (25.7, 36.4), turned to 0 degrees
- moved U$3 17.4 mm to (46.7, 37.2)
- moved J1 17.3 mm to (68.4, 41.4)
- moved J2 17.2 mm to (24.7, 45.2)
Connections:
- new net ADC_FOTO: U$6.10
- new net CE_RADIO: U$7.1
- new net CS_RADIO: U$7.2
- new net DIR_DRIVER: U$6.1
- new net IRQ_RADIO: U$7.3
- new net LATCH_SR: U$6.5
- new net MISO_RADIO: U$7.5
- new net MISO_SR: U$6.8
- new net MOSI_RADIO: U$7.4
- new net MOSI_SR: U$6.9
- new net OE_SR: U$6.6
- new net RX1_BLE: U$6.4
- new net RX2_GPS: U$7.8
- new net SCK_RADIO: U$7.6
- new net SCK_SR: U$6.7
- new net STEP_DRIVER: U$6.2
- new net SV: U$6.11
- new net SW_WMP: U$7.9
- new net TX1_BLE: U$6.3
- new net TX2_GPS: U$7.7
- net 3V3: now also U$6.13
- net GND: now also U$6.12
Routing:
- net GND: track 0.00 -> 147.0 mm, vias 0 -> 2
- net 3V3: track 0.00 -> 120.8 mm, vias 0 -> 3
- net LED1: track 0.00 -> 4.66 mm
- net LED2: track 0.00 -> 4.07 mm
- net ATN_RADIO: track 0.00 -> 2.26 mm
- net RF-IN: track 0.00 -> 2.10 mm

Commit message: кцуенгшщозлдх
Parts:
- added U$8: PBS_SMD_X13, UNKNOWN-2024:PBD_SMD_X13
- moved U$2 9.75 mm to (50.4, 69.0), turned to 0 degrees
Connections:
- removed net CE: U$2.P$2
- removed net CSN: U$2.P$3
- removed net IRQ: U$2.P$7
- removed net MISO: U$2.P$6
- removed net MOSI: U$2.P$5
- removed net RX: U$1.P$2
- removed net SCK: U$2.P$4
- removed net SV: U$6.11
- removed net SW: U$3.SW
- removed net TX: U$1.P$3
- net 3V3: now also U$8.13
- net 5V: now also U$6.11, U$8.11
- net ADC_FOTO: now also U$8.10
- net CE_RADIO: now also U$2.P$2
- net CS_RADIO: now also U$2.P$3
- net DIR_DRIVER: now also U$8.1
- net GND: now also U$8.12
- net IRQ_RADIO: now also U$2.P$7
- net LATCH_SR: now also U$8.5
- net MISO_RADIO: now also U$2.P$6
- net MISO_SR: now also U$8.8
- net MOSI_RADIO: now also U$2.P$5
- net MOSI_SR: now also U$8.9
- net OE_SR: now also U$8.6
- net RX1_BLE: now also U$8.4
- net RX2_GPS: now also U$1.P$2
- net SCK_RADIO: now also U$2.P$4
- net SCK_SR: now also U$8.7
- net STEP_DRIVER: now also U$8.2
- net SW_WMP: now also U$3.SW
- net TX1_BLE: now also U$8.3
- net TX2_GPS: now also U$1.P$3
Routing:
- net 5V: track 0.00 -> 37.7 mm
- net SW_WMP: track 0.00 -> 32.5 mm
- net SCK_RADIO: track 0.00 -> 28.1 mm
- net MOSI_RADIO: track 0.00 -> 19.0 mm
- net CS_RADIO: track 0.00 -> 16.3 mm
- net MISO_RADIO: track 0.00 -> 15.3 mm, vias 0 -> 2
- net IRQ_RADIO: track 0.00 -> 15.1 mm, vias 0 -> 2
- net RX2_GPS: track 0.00 -> 15.0 mm
- net CE_RADIO: track 0.00 -> 13.1 mm
- net GND: track 147.0 -> 157.4 mm
- net TX2_GPS: track 0.00 -> 8.97 mm
- net 3V3: track 120.8 -> 126.0 mm

Commit message: горншлщ90зд-жхэзжотрм с
Parts:
- moved U$8 57.3 mm to (75.0, 52.0), flipped to the bottom, turned to 270 degrees
Connections:
- net 3V3: now also U$8.1; no longer U$8.13
- net 5V: now also U$8.3; no longer U$8.11
- net ADC_FOTO: now also U$8.4; no longer U$8.10
- net DIR_DRIVER: now also U$8.13; no longer U$8.1
- net GND: now also U$8.2; no longer U$8.12
- net LATCH_SR: now also U$8.9; no longer U$8.5
- net MISO_SR: now also U$8.6; no longer U$8.8
- net MOSI_SR: now also U$8.5; no longer U$8.9
- net OE_SR: now also U$8.8; no longer U$8.6
- net RX1_BLE: now also U$8.10; no longer U$8.4
- net STEP_DRIVER: now also U$8.12; no longer U$8.2
- net TX1_BLE: now also U$8.11; no longer U$8.3
Routing:
- net MISO_RADIO: track 15.3 -> 37.5 mm
- net IRQ_RADIO: track 15.1 -> 31.6 mm
- net 3V3: track 126.0 -> 130.5 mm
- net TX1_BLE: track 0.00 -> 4.22 mm, vias 0 -> 1
- net LATCH_SR: track 0.00 -> 3.69 mm, vias 0 -> 1
- net MISO_SR: track 0.00 -> 3.62 mm, vias 0 -> 1
- net ADC_FOTO: track 0.00 -> 3.49 mm, vias 0 -> 1
- net MOSI_SR: track 0.00 -> 3.33 mm, vias 0 -> 1
- net RX1_BLE: track 0.00 -> 3.30 mm, vias 0 -> 1
- net OE_SR: track 0.00 -> 3.15 mm, vias 0 -> 1
- net STEP_DRIVER: track 0.00 -> 3.15 mm, vias 0 -> 1
- net DIR_DRIVER: track 0.00 -> 3.13 mm, vias 0 -> 1
- net SCK_SR: track 0.00 -> 3.09 mm, vias 0 -> 1
- net 5V: track 37.7 -> 39.3 mm, vias 0 -> 1
- net GND: track 157.4 -> 158.6 mm, vias 2 -> 3
- added copper zone on layer 16, net гнд

Commit message: плата рпарпарпараарпарпарпааарпарпарпауекуекуекусруркра
Parts:
- added LED1, LED2: (no value), led:CHIPLED_0603
- added R1, R2: (no value), rcl:R0603
- moved J1 0.36 mm to (68.6, 41.1)
Connections:
- removed net LED1: U$3.LED1, U$4.2
- removed net LED2: U$3.LED2, U$5.2
- new net N$1: LED1.C, R1.2
- new net N$2: LED2.C, R2.2
- new net N$3: LED1.A, U$4.2
- new net N$4: LED2.A, U$5.2
- new net N$5: R2.1, U$3.LED2
- new net N$6: R1.1, U$3.LED1
Routing:
- net GND: track 158.6 -> 166.5 mm
- net LED1: track 4.66 -> 0.00 mm
- net MOSI_RADIO: track 19.0 -> 23.4 mm
- net LED2: track 4.07 -> 0.00 mm
- net SW_WMP: track 32.5 -> 35.1 mm
- net 5V: track 39.3 -> 40.9 mm
- net SCK_RADIO: track 28.1 -> 29.5 mm
- net 3V3: track 130.5 -> 129.4 mm
- net TX2_GPS: track 8.97 -> 9.71 mm
- added copper zone on layer 1, net GND
- added copper zone on layer 16, net GND
- removed copper zone on layer 16, net гнд

Commit message: sdfghgfds
Parts:
- added C1: (no value), rcl:C0603
- added C2: ECAPECAP220, CanCubeSat:ECAP220-CMD
- moved R1 0.36 mm to (25.1, 29.7)
- moved R2 0.32 mm to (26.1, 40.0)
- moved LED2 0.30 mm to (24.0, 40.1)
- moved LED1 0.28 mm to (25.0, 31.5)
Connections:
- net 3V3: no longer U$3.3.3V
- net 5V: now also C1.2, C2.P$1
- net GND: now also C1.1, C2.P$2
Routing:
- net 3V3: track 129.4 -> 91.5 mm, vias 3 -> 4
- net 5V: track 40.9 -> 55.7 mm
- net SW_WMP: track 35.1 -> 25.9 mm, vias 0 -> 2
- net GND: track 166.5 -> 160.7 mm, vias 3 -> 2
- net N$4: track 0.00 -> 3.69 mm
- net N$6: track 0.00 -> 2.58 mm
- net N$5: track 0.00 -> 2.44 mm
- net N$2: track 0.00 -> 2.10 mm
- net N$1: track 0.00 -> 1.80 mm
- net N$3: track 0.00 -> 1.60 mm

Commit message: ывавп лыл
Parts:
- C1: value (none) -> 100nF
- C2: value ECAPECAP220 -> 220uF
- J1: value U.FL-R-SMT-1_10_ -> IPX-RADIO
- J2: value U.FL-R-SMT-1_10_ -> IPX-ANT
- LED1: value (none) -> AMP1
- LED2: value (none) -> AMP2
- R1, R2: value (none) -> 2k
- renumbered U$1 to GPS-NEO7M, U$2 to NRF24LO1, U$3 to XQ-02A, U$4 to ROTATE1, U$5 to ROTATE2
Connections:
- removed net ATN_RADIO: J2.3, XQ-02A.ATN
- new net ANT_RADIO: J2.3, XQ-02A.ANT
Routing:
- net ATN_RADIO: track 2.26 -> 0.00 mm
- net ANT_RADIO: track 0.00 -> 2.26 mm
- net 3V3: track 91.5 -> 91.4 mm, vias 4 -> 3

Commit message: Платы вроде готовы
Connections:
- net DIR_DRIVER: now also U$6.2, U$8.12; no longer U$6.1, U$8.13
- net STEP_DRIVER: now also U$6.1, U$8.13; no longer U$6.2, U$8.12
Routing:
- net 5V: track 55.7 -> 54.5 mm
- net DIR_DRIVER: track 3.13 -> 4.10 mm
- net OE_SR: track 3.15 -> 4.01 mm
- net SCK_SR: track 3.09 -> 3.94 mm
- net STEP_DRIVER: track 3.15 -> 3.93 mm
- net MOSI_SR: track 3.33 -> 4.01 mm
- net MISO_RADIO: track 37.2 -> 37.9 mm
- net RX1_BLE: track 3.30 -> 3.92 mm
- net GND: track 160.7 -> 161.2 mm
Other:
- board text added: "3V3"
- board text added: "5V"
- board text added: "CE"
- board text added: "CS"
- board text added: "DIR"
- board text added: "FOTO"
- board text added: "GND"
- board text added: "IRQ"
- board text added: "LATCH"
- board text added: "MISO"
- board text added: "MOSI"
- board text added: "OE"
- board text added: "RX1"
- board text added: "RX2"
- board text added: "SCK"
- board text added: "STEP"
- board text added: "SW"
- board text added: "TX1"
- board text added: "TX2"
